File: shields/tv/tv.sch (EAGLE design)
At the start: 20 parts, among them U1 VS23S010D-L, U2 OPENMV3, U3 TX5813, X1 uFL, X3 736880-49, Y1 28.63636MHZ

Commit message: add pdf
Other:
- note added: "5.8G Transmitter"
- note added: "Copyright (c) 2019 kaizhi <kaizhi@singtown.com>"
- note added: "NTSC Generate"
- note removed: "Copyright (c) 2013 Ibrahim Abd Elkader <i.abdalkader@gmail.com>"
Changed lines of the file:
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@@
 <wire x1="314.96" y1="231.14" x2="314.96" y2="0" width="0.1524" layer="94"/>
 <wire x1="198.12" y1="231.14" x2="314.96" y2="231.14" width="0.1524" layer="94"/>
-<wire x1="198.12" y1="231.14" x2="198.12" y2="0" width="0.1524" layer="94"/>
+<wire x1="198.12" y1="231.14" x2="198.12" y2="121.92" width="0.1524" layer="94"/>
+<wire x1="198.12" y1="121.92" x2="198.12" y2="0" width="0.1524" layer="94"/>
 <wire x1="314.96" y1="0" x2="198.12" y2="0" width="0.1524" layer="94"/>
 <wire x1="198.12" y1="0" x2="0" y2="0" width="0.1524" layer="94"/>
 <text x="203.2" y="223.52" size="5.08" layer="150" ratio="10">OpenMV</text>
-<text x="2.54" y="15.24" size="3.81" layer="150">Copyright (c) 2013 Ibrahim Abd Elkader &lt;i.abdalkader@gmail.com&gt;</text>
+<text x="2.54" y="15.24" size="3.81" layer="150">Copyright (c) 2019 kaizhi &lt;kaizhi@singtown.com&gt;</text>
 <text x="2.54" y="10.16" size="3.81" layer="150">This work is licensed under the Creative Commons Attribution-ShareAlike 3.0 License.</text>
 <text x="2.54" y="5.08" size="3.81" layer="150">To view a copy of this license, visit http://creativecommons.org/licenses/by-sa/3.0/</text>
@@
 <wire x1="198.12" y1="231.14" x2="0" y2="231.14" width="0.1524" layer="94"/>
 <wire x1="0" y1="231.14" x2="0" y2="0" width="0.1524" layer="94"/>
+<wire x1="0" y1="121.92" x2="198.12" y2="121.92" width="0.1524" layer="94"/>
+<text x="5.08" y="223.52" size="5.08" layer="150" ratio="10">NTSC Generate</text>
+<text x="5.08" y="111.76" size="5.08" layer="150" ratio="10">5.8G Transmitter</text>
 </plain>
 <instances>
