File: openmv4/sensors/OV5640/OV5640.sch (EAGLE design)
At the start: 14 parts, among them U1 OV5640-A71A, U4 ADP150AUJZ-2.8-R7

Commit message: Updated OV5640 circuit
Parts:
- removed L2: BEAD, heka:BEAD
- removed U$3: DF12-36-DP, DF12:DF12-36-DP
- removed U4: ADP150AUJZ-2.8-R7, leptonCustom:ADP150TSOT-5
- added C10, C11, C12, C9: 0.1uF, sfe:CAP0402-CAP
- added C13, C14: 1uF, sfe:CAP0402-CAP
- added C15, C16, C17: 10uF, sfe:CAP0402-CAP
- added U2: ME6211C28M5G, leptonCustom:ADP150TSOT-5
- added U3: ME6211C15M5G, leptonCustom:ADP150TSOT-5
- added X1: DF12-36-DP, DF12:DF12-36-DP
- C1, C2: value 1 uF -> 1uF; device SparkFun-Capacitors:CAP0402-CAP -> sfe:CAP0402-CAP
- C3: value 0.1uF -> 1uF
- L1: value BEAD -> MPZ1608S181ATAH0
Connections:
- net N$1 renamed VN
- net N$3 renamed VH
- removed net DVDD: C4.2, C5.2, U1.DVDD, U1.DVDD@1, U1.DVDD@2, U1.DVDD@3, U1.DVDD@4, U1.DVDD@5, U1.DVDD@6
- removed net PVDD: L2.2, U1.PVDD
- new net 1V5: C12.2, C14.2, C17.2, C4.2, C5.2, U1.DVDD, U1.DVDD@1, U1.DVDD@2, U1.DVDD@3, U1.DVDD@4, U1.DVDD@5, U1.DVDD@6, U1.EVDD, U3.VOUT
- net 2V8: now also C16.2, C2.2, U2.VOUT; no longer C2.1, L2.1, U1.EVDD, U4.VOUT
- net AVDD: now also C10.2, C11.2, C15.2, C9.2, U1.PVDD
- net DCMI_CLK: now also X1.12; no longer U$3.12
- net DCMI_D0: now also X1.31; no longer U$3.31
- net DCMI_D1: now also X1.29; no longer U$3.29
- net DCMI_D2: now also X1.35; no longer U$3.35
- net DCMI_D3: now also X1.28; no longer U$3.28
- net DCMI_D4: now also X1.26; no longer U$3.26
- net DCMI_D5: now also X1.33; no longer U$3.33
- net DCMI_D6: now also X1.24; no longer U$3.24
- net DCMI_D7: now also X1.22; no longer U$3.22
- net DCMI_FSIN: now also U1.FREX, X1.23; no longer U$3.23
- net DCMI_HSYNC: now also X1.18; no longer U$3.18
- net DCMI_PCLK: now also X1.14; no longer U$3.14
- net DCMI_PWDN: now also X1.25; no longer U$3.25
- net DCMI_RST: now also X1.21; no longer U$3.21
- net DCMI_VSYNC: now also X1.16; no longer U$3.16
- net GND: now also C1.1, C10.1, C11.1, C12.1, C13.1, C14.1, C15.1, C16.1, C17.1, C2.1, C9.1, U2.GND, U3.GND, X1.19, X1.27, X1.5; no longer C1.2, C2.2, U$3.19, U$3.27, U$3.5, U4.GND
- net I2C1_SCL: now also X1.32; no longer U$3.32
- net I2C1_SDA: now also X1.34; no longer U$3.34
- net RSVD1: now also X1.1; no longer U$3.1
- net RSVD2: now also X1.3; no longer U$3.3
- net RSVD3: now also X1.7; no longer U$3.7
- net RSVD4: now also X1.9; no longer U$3.9
- net RSVD5: now also X1.6; no longer U$3.6
- net RSVD6: now also X1.8; no longer U$3.8
- net SPI3_MISO: now also X1.15; no longer U$3.15
- net SPI3_MOSI: now also X1.17; no longer U$3.17
- net SPI3_SCLK: now also X1.13; no longer U$3.13
- net SPI3_SSEL: now also X1.11; no longer U$3.11
- net VCC: now also C1.2, C13.2, U2.EN, U2.VIN, U3.EN, U3.VIN, X1.10, X1.2, X1.20, X1.30, X1.36; no longer C1.1, U$3.10, U$3.2, U$3.20, U$3.30, U$3.36, U4.EN, U4.VIN
Other:
- note added: "CONNECTOR"
- note added: "POWER"
- moved on the sheet: C1, C2, C3, C4, C5, C6, C7, C8, L1, U1
