File: openmv4/base-alt/base-alt.brd (EAGLE design)
At the start: 35.6 x 44.5 mm, 63 parts, among them M1 9774030243R, M2 9774030243R, Q1 BSS138, Q2 Si2301BDS, U2 STM32H743XIH6, U5 TPS731XX, U8 PAM2305AABADJ, X1 MF-CON-MICROUSB-RIGHT, X2 USD-1040310811, X3 DF12-36-DS, X4 S2B-PH-K-S(LF)(SN), Y1 7S-12.000MAHE-T

Commit message: PureEngineering Updates
Routing:
- net GND: track 74.0 -> 81.3 mm, vias 62 -> 61
- net VCC: track 71.8 -> 74.1 mm
