File: openmv4/plus-alt/plus-alt.sch (EAGLE design)
At the start: 76 parts, among them M1 9774030243R, M2 9774030243R, Q1 BSS138, Q2 AO3401, U1 W25Q256JVEIQ_TR, U2 *, U3 ME6211C33M5G, U4 PAM2305AABADJ, U5 USBLC6-2, X1 MF-CON-MICROUSB-RIGHT, X2 USD-1040310811, X3 DF12-36-DS, X4 S2B-PH-K-S(LF)(SN), Y1 12M

Commit message: Fixed QSPI pins
Connections:
- net FLASH_IO0: now also U2A.PF8; no longer U2A.PF9
- net FLASH_IO1: now also U2A.PF9; no longer U2A.PF8
