File: openmv-mp/openmv-mp.sch (EAGLE design)
At the start: 44 parts, among them J1 503398-1892, M1 9774030243R, M2 9774030243R, Q1 BSS138, Q2 Si2301BDS, U1 OSD32MP157C-512M-BAA, X3 DF12-36-DS, X4 S2B-PH-K-S(LF)(SN), X6 MF-CON-MICROUSB-RIGHT

Commit message: Update design
Parts:
- removed C24: 10uF, sfe:CAP0402-CAP
- removed C25, C26: 0.01uF, sfe:CAP0402-CAP
- removed C35: 100uF, sfe:CAP_POL1206
- removed JP4, JP6: (no value), pinhead:PINHD-2X8
- removed Q2: Si2301BDS, sfe:MOSFET-PCHANNELSMD
- removed R42: 10K, sfe:RESISTOR0402-RES
- removed RN1: 220R, resistor-dil:4R-NEXBV8V
- removed RN2, RN5: 10K, resistor-dil:4R-NEXBV8V
- removed U$10, U$9: SWITCHKMS221G, mux:SWITCHKMS221G
- removed X4: S2B-PH-K-S(LF)(SN), adafruit-updated:JST_2PIN-THM-RA
- removed X6: MF-CON-MICROUSB-RIGHT, MF_Connectors:USB_MICRO_RIGHT
- added ANT1: 2450AT18B100E, 2450AT18B100E:2450AT18B100E
- added C11, C13, C16, C22, C3, C9: 0.1uF, sfe:CAP0402-CAP
- added C12: 10uF, sfe:CAP0402-CAP
- added C15, C2, C21: 4.7uF, sfe:CAP0402-CAP
- added C18: 2.2uF, sfe:CAP0402-CAP
- added C19: 1uF, sfe:CAP0402-CAP
- added C20, C5, C6, C7, C8: 47uF, sfe:CAP0805
- added C4: 220uF, sfe:CAP1206
- added D2: ESDALC6V1-1U2, esd:ESDALC6V1-1U2
- added D4, D5, D6: ESDA7P120-1U1M, esd:ESDA7P120-1U1M
- added JP1, JP2: (no value), pinhead:PINHD-2X8
- added L1, L2: MPZ1608S101ATAH0, sfe:INDUCTOR0402
- added L3: 2.2uH, sfe:INDUCTOR0603
- added R10, R11, R7, R8: 47K, sfe:RESISTOR0402-RES
- added R16, R27, R28, R31, R5, R6: 10K, sfe:RESISTOR0402-RES
- added R17, R23: 23.7K, sfe:RESISTOR0402-RES
- added R18, R24: 5K, sfe:RESISTOR0402-RES
- added R19, R20, R21, R22: 220R, sfe:RESISTOR0402-RES
- added R25: 10R, sfe:RESISTOR0402-RES
- added R26: 56K, sfe:RESISTOR0402-RES
- added R29, R30: 2.2K, sfe:RESISTOR0402-RES
- added SJ1: SOLDERJUMPERNO, sfe:SOLDERJUMPERNO
- added TP1, TP2: TPTP10R, testpad:TPTP10R
- added U2, U3: ECMF02-2AMX6, esd:ECMF02-2AMX6
- added U4: LBEE5KL1DX-TEMP, LBEE5KL1DX-TEMP:LBEE5KL1DX-TEMP
- added U5: EMIF06-MSD02N16, esd:EMIF06-MSD02N16
- added U6: TPS2121, mux:TPS2121
- added U7: VL53L1X, SparkFun-Sensors:VL53L1XSMD
- added X1: DF12-36-DS, DF12:DF12-36-DS
- added X2: S2B-PH-K-S(LF)(SN), adafruit-updated:JST_2PIN-THM-RA
- C1: value 22uF -> 4.7uF; device sfe:CAP0805 -> sfe:CAP0402-CAP
- C10, C17: value 0.1uF -> 10uF
- C14: value 47uF -> 1.2pF; device sfe:CAP_POL1206 -> sfe:CAP0402-CAP
- D1: value SDM2U20SD3-7 -> ESDA7P120-1U1M; device sfe:DIODESOD -> esd:ESDA7P120-1U1M
- D3: value SDM2U20SD3-7 -> ESDALC6V1-1U2; device sfe:DIODESOD -> esd:ESDALC6V1-1U2
- J1: value 503398-1892 -> (none); device 503398-1892:503398-1892 -> PP_Connectors:USB_TYPE-C_105450-0101
- L4: value MPZ1608S181ATAH0 -> 3.3nH
- L5: value MPZ1608S181ATAH0 -> 2.7nH
- R1: value 10R -> 10K
- R12, R13: value 22R -> 5K1/10%
- R14: value 22R -> 4.7K
- R15: value 10K -> 4.7K
- R3, R4: value 4.7K -> 10K
- R9: value 10K -> 47K
- X3: value DF12-36-DS -> 503398-1892; device DF12:DF12-36-DS -> 503398-1892:503398-1892
Connections:
- removed net 3V3_OUT: D1.C, JP4.15, JP4.16
- removed net DAC2: JP4.13, U1B.PA5
- removed net N$35: R12.2, X6.D-
- removed net N$37: R14.2, X6.ID
- removed net N$38: L5.1, X6.SLD
- removed net OTG_HS_DN: R12.1, U1D.USB_DM2
- removed net OTG_HS_DP: R13.1, U1D.USB_DP2
- removed net OTG_HS_ID: R14.1, U1B.PA10
- removed net SDMMC2_D4: U1B.PA8
- removed net SDMMC2_D5: U1B.PA9
- removed net SDMMC2_D6: U1C.PE5
- removed net SDMMC2_D7: U1B.PD3
- removed net SPI6_MISO: JP6.9, U1C.PG12
- removed net SPI6_MOSI: JP6.11, U1C.PG14
- removed net SPI6_SCLK: JP6.7, U1C.PG13
- removed net TIM2_CH2: JP4.10, U1B.PA1
- removed net VDDA: X3.4
- new net ANA0: JP2.9, U1D.ANA0
- new net BT_DEV_WAKE: U1C.PZ7, U4.BT_DEV_WAKE
- new net BT_HOST_WAKE: U1C.PZ3, U4.BT_HOST_WAKE
- new net BT_REG_ON: U1C.PZ6, U4.BT_REG_ON
- new net CC1: D2.C, J1.CC1, R12.2, U1C.PF13
- new net CC2: D3.C, J1.CC2, R13.2, U1C.PF14
- new net DN: J1.D-, U3.DP_I
- new net DP: J1.D+, U3.DM_I
- new net FDCAN2_RX: JP1.12, U1B.PB5
- new net FDCAN2_TX: JP1.10, U1B.PB13
- new net HDM: JP1.4, U2.DP_O
- new net HDP: JP1.2, U2.DM_O
- new net I2C6_SCL: R30.2, U1B.PD1, U7.SCL
- new net I2C6_SDA: R29.2, U1B.PD0, U7.SDA
- new net N$11: TP2.TP, U1A.PMIC_LDO5
- new net N$12: U5.DAT3_EX, X3.CD/DAT3^2
- new net N$13: U5.DAT2_EX, X3.DAT2
- new net N$2: R4.2, U1A.HSE_OSC_OE
- new net N$30: U5.DAT1_EX, X3.DAT1
- new net N$31: U5.DAT0_EX, X3.DAT0
- new net N$32: U5.CLK_EX, X3.CLK
- new net N$33: U5.CMD_EX, X3.CMD
- new net N$39: R23.2, R24.1, U6.OV1
- new net N$40: C19.1, U6.SS
- new net N$41: R17.2, R18.1, U6.OV2
- new net N$42: R26.1, U6.ILIM
- new net N$44: C14.1, L4.1, L5.2
- new net N$45: ANT1.1, L4.2
- new net N$46: C14.2, U4.ANT
- new net N$47: C15.1, L3.2, U4.VIN_LDO
- new net N$48: L3.1, U4.SR_VLX
- new net N$7: SJ1.2, U1A.EEPROM_WP
- new net PWR_ST: R27.2, U1B.PA7, U6.ST
- new net SWC: JP2.5, U1D.JTCK-SWCLK
- new net SWD: JP2.7, U1D.JTMS-SWDIO
- new net SWO: JP2.3, U1D.JTDO-TRACESWO
- new net USART2_CTS: U1B.PD3, U4.!BT_UART_RTS_N
- new net USART2_RTS: U1B.PD4, U4.!BT_UART_CTS_N
- new net USART2_RX: U1B.PD6, U4.BT_UART_TXD
- new net USART2_TX: U1B.PD5, U4.BT_UART_RXD
- new net USART3_RX: JP2.13, U1B.PD9
- new net USART3_TX: JP2.11, U1B.PD8
- new net USBD_DM: U1D.USB_DM2, U3.DP_O
- new net USBD_DP: U1D.USB_DP2, U3.DM_O
- new net VLX_IRQ: R31.2, U1B.PA2, U7.!INT
- new net VLX_SHUT: R28.2, U1B.PA5, U7.!SHUT
- new net VSSA: U1D.VREF-, U1D.VSSA
- new net WL_HOST_WAKE: U1B.PD7, U4.WL_GPIO_0_HOST_WAKE
- new net WL_LPO_32: TP1.TP, U1C.PI8
- new net WL_REG_ON: U1C.PH4, U4.WL_REG_ON
- net 3V3: now also C16.1, C17.1, C18.1, C21.1, C22.1, C5.1, C6.1, C7.1, C8.1, C9.1, D1.C, JP1.15, JP1.16, LED3.A, R1.1, R10.2, R11.2, R14.1, R2.1, R27.1, R28.1, R29.1, R30.1, R31.1, R6.1, R7.2, R8.2, R9.2, U1D.VREF+, U4.VBAT, U4.VIO, U5.RDATA_VCC, U5.VCC, U7.VCC, X1.10, X1.2, X1.20, X1.30, X1.36, X1.4, X3.VDD; no longer C1.1, C10.1, C14.+, C35.+, D1.A, J1.VDD, LED2.A, R4.1, R42.1, RN2A.2, RN2B.2, RN2C.2, RN2D.2, RN5A.2, RN5B.2, RN5C.2, RN5D.2, X3.10, X3.2, X3.20, X3.30, X3.36
- net BOOT: now also JP2.4, R6.2; no longer JP6.4, RN5D.1
- net DAC1: now also JP1.13; no longer JP4.12
- net DCMI_CLK: now also X1.12; no longer X3.12
- net DCMI_D0: now also X1.31; no longer X3.31
- net DCMI_D1: now also X1.29; no longer X3.29
- net DCMI_D10: now also X1.7; no longer X3.7
- net DCMI_D11: now also X1.9; no longer X3.9
- net DCMI_D2: now also X1.35; no longer X3.35
- net DCMI_D3: now also X1.28; no longer X3.28
- net DCMI_D4: now also X1.26; no longer X3.26
- net DCMI_D5: now also X1.33; no longer X3.33
- net DCMI_D6: now also X1.24; no longer X3.24
- net DCMI_D7: now also X1.22; no longer X3.22
- net DCMI_D8: now also X1.3; no longer X3.3
- net DCMI_D9: now also U1C.PI2, X1.1; no longer U1C.PH7, X3.1
- net DCMI_FSIN: now also JP2.6, X1.23; no longer JP6.6, X3.23
- net DCMI_HSYNC: now also X1.18; no longer X3.18
- net DCMI_PCLK: now also U1B.PA6, X1.14; no longer U1B.PC2, X3.14
- net DCMI_PWDN: now also X1.25; no longer X3.25
- net DCMI_RST: now also X1.21; no longer X3.21
- net DCMI_VSYNC: now also X1.16; no longer X3.16
- net EEPROM_WP: now also SJ1.1, U1C.PI6; no longer U1A.EEPROM_WP
- net GND: now also C1.1, C11.2, C12.2, C13.2, C15.2, C16.2, C18.2, C19.2, C2.1, C20.2, C21.2, C22.2, C3.2, C4.2, C5.2, C6.2, C7.2, C8.2, C9.2, D1.A, D2.A, D3.A, D4.A, D5.A, D6.A, J1.GND, JP2.15, JP2.16, L2.2, L5.1, R12.1, R13.1, R16.1, R18.2, R24.2, R26.2, R4.1, R5.2, U2.GND, U3.GND, U4.GND, U4.GND_(SR_PVSS), U4.LPO_IN_(32KHZ), U5.GND, U6.CP2, U6.GND, U6.PR1, U7.GND, X1.19, X1.27, X1.5, X2.1, X3.SHIELD, X3.VSS; no longer C1.2, C14.-, C24.2, C25.2, C26.2, C35.-, J1.SHIELD, J1.VSS, JP6.15, JP6.16, L5.2, R2.1, R9.1, U$10.1, U$9.1, X3.19, X3.27, X3.5, X4.1, X6.GND
- net I2C2_SCL: now also JP1.9; no longer JP4.9
- net I2C2_SDA: now also JP1.11; no longer JP4.11
- net I2C5_SCL: now also R14.2, X1.32; no longer R3.2, X3.32
- net I2C5_SDA: now also R15.2, X1.34; no longer R4.2, X3.34
- net LED_B: now also R20.1, U1C.PE10; no longer RN1B.2, U1C.PZ3
- net LED_G: now also R21.1, U1C.PE9; no longer RN1C.2, U1C.PZ4/PMIC_SCL
- net LED_IR: now also R22.1; no longer RN1D.2
- net LED_R: now also R19.1, U1C.PE8; no longer RN1A.2, U1C.PZ6
- net N$10: now also LED2.C, R25.2; no longer LED3.C, R1.2
- net N$14: now also R25.1; no longer R1.1
- net N$17: now also LED2.A, LED3.C; no longer LED2.C, LED3.A
- net N$34: now also D4.C, J1.VBUS, L1.1; no longer L4.1, X6.5V
- net N$36: now also R5.1, U1A.BOOT1; no longer R13.2, X6.D+
- net N$4: now also J1.SHLD, L2.1; no longer JP6.3
- net N$5: now also R16.2, R22.2; no longer R2.2, RN1D.1
- net N$6: now also R20.2; no longer RN1B.1
- net N$8: now also R19.2; no longer RN1A.1
- net N$9: now also R21.2; no longer RN1C.1
- net NRST: now also JP2.2, R1.2; no longer C26.1, JP6.2, R42.2, U$10.2
- net PONKEY: now also JP2.1, R3.2; no longer C25.1, JP6.1, R15.2, U$9.2
- net RSVD5: now also X1.8; no longer X3.8
- net RSVD6: now also X1.6; no longer X3.6
- net SDMMC1_CK: now also U5.CLK_IN; no longer J1.CLK
- net SDMMC1_CMD: now also U5.CMD_IN; no longer J1.CMD, RN2C.1
- net SDMMC1_D0: now also U5.DAT0_IN; no longer J1.DAT0, RN2B.1
- net SDMMC1_D1: now also U5.DAT1_IN; no longer J1.DAT1, RN5B.1
- net SDMMC1_D2: now also U5.DAT2_IN; no longer J1.DAT2, RN5A.1
- net SDMMC1_D3: now also U5.DAT3_IN; no longer J1.CD/DAT3^2, RN2D.1
- net SDMMC2_CK: now also U4.SDIO_CLK
- net SDMMC2_CMD: now also R7.1, U4.SDIO_CMD
- net SDMMC2_D0: now also R8.1, U4.SDIO_DATA_0
- net SDMMC2_D1: now also R9.1, U4.SDIO_DATA_1
- net SDMMC2_D2: now also R10.1, U4.SDIO_DATA_2
- net SDMMC2_D3: now also R11.1, U4.SDIO_DATA_3
- net SPI2_MISO: now also JP1.3, U1B.PC2; no longer JP4.3, U1C.PI2
- net SPI2_MOSI: now also JP1.1; no longer JP4.1
- net SPI2_NSS: now also JP1.7; no longer JP4.7
- net SPI2_SCLK: now also JP1.5; no longer JP4.5
- net SPI3_MISO: now also X1.15; no longer X3.15
- net SPI3_MOSI: now also U1B.PA8, X1.17; no longer U1B.PD6, X3.17
- net SPI3_SCLK: now also X1.13; no longer X3.13
- net SPI3_SSEL: now also X1.11; no longer X3.11
- net SPI6_NSS: no longer JP6.5
- net TIM4_CH1: now also JP2.12; no longer JP6.12
- net TIM4_CH2: now also JP2.10; no longer JP6.10
- net TIM4_CH3: now also JP2.8; no longer JP6.8
- net UART4_RX: now also JP1.6; no longer JP4.6
- net UART4_TX: now also JP1.8, R2.2; no longer JP4.8, RN2A.1
- net USBH_DM: now also U2.DP_I; no longer JP4.4
- net USBH_DP: now also U2.DM_I; no longer JP4.2
- net USD_DETECT: now also U5.WP/CD, X3.DETECT_SWITCH; no longer J1.DETECT_SWITCH, RN5C.1
- net VBAT: now also C12.1, C13.1, D6.C, JP2.14, R17.1, U6.IN2, X2.2; no longer D3.A, JP6.13, JP6.14, Q2.G, R9.2, X4.2
- net VBUS: now also C10.1, C11.1, L1.2, R23.1, U6.IN1; no longer C17.1, C24.1, L4.2, Q2.D, U1A.PMIC_VBUSOTG, U1D.OTG_VBUS
- net VBUS_SW: now also C3.1, C4.1, D5.C, JP1.14; no longer JP4.14
- net VIN: now also C1.2, C2.2, C20.1, U6.OUT; no longer D3.C, Q2.S
Other:
- note added: "!"
- note added: "* Length match DCMI signals"
- note added: "* Length match SD signals."
- note added: "* Length math SD signals."
- note added: "* No vias under socket"
- note added: "* PMIC I2C4 * DO NOT USE"
- note added: "* Tune Ant matching network"
- note added: "* Use 50ohm feed line"
- note added: "0"
- note added: "BOOT0"
- note added: "BOOT1"
- note added: "BOOT2"
- note added: "Copyright (c) 2020 OpenMV <openmv@openmv.io>"
- note added: "MODE"
- note added: "N/A"
- note added: "OSD32MP1 SiP"
- note added: "POWER MUX"
- note added: "Pulldown may be required"
- note added: "SD"
- note added: "USB"
- note added: "USBC"
- note added: "WiFi/Bluetooth"
- note removed: "Copyright (c) 2018 OpenMV <openmv@openmv.io>"
- note removed: "MPU"
- note removed: "USB & VIN"
- moved on the sheet: C1, C10, C17, L4, L5, LED1, LED2, LED3, Q1, R1, R12, R13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
