File: openmv4/pro/pro-base.brd (EAGLE design)
At the start: 35.6 x 44.5 mm, 176 parts, among them J2 SAMTEC_FTSH-105-01-F-DVSAMTEC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, J6 RSP-122811-01, M1 9774030243R, M2 9774030243R, Q1 BSS138, Q2 AO3401, U1 W25Q256JVEIQ_TR, U10 STM32H743IIK6, U11 TEXAS_INSTRUMENTS_BQ24072TRGT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, U12 MICROCHIP_ATECC608A-SSHDA-BMI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, U14 IS42S32800, U2 EMIF06-MSD02N16, U3 ME6211C18M5G, U4 PAM2305AABADJ, U5 LSM6DS3TR-C, U6 MICROCHIP_USB3320C-EZK-TRMICR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, U7 LBEE5KL1DX-TEMP, U9 VL53L5CX, X2 USD-1040310811, X3 DF12-36-DS, X4 S2B-PH-K-S(LF)(SN), Y0 SITIME_SIT1533AI-H4-DCC-32.76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, Y1 DSC1001BI1-024.0000

Commit message: Update pro schematics
Parts:
- added D26: GREEN, SparkFun-LED:LED-0603
- added JP3, JP4: JUMPER-SMT_2_NC_PASTE_SILK, SparkFun-Jumpers:SMT-JUMPER_2_NC_PASTE_SILK
- added R46: 1.5K, sfe:0402-RES
- moved R29 0.40 mm to (14.4, 6.40)
- moved C53 0.40 mm to (14.4, 3.65)
Connections:
- new net N$1: D26.A, R46.1
- new net N$11: JP4.1, R33.2
- new net N$12: JP3.1, R46.2
- new net N$9: D26.C, U11.7
- net OUT: now also JP3.2, JP4.2; no longer R33.2
Changed lines of the file:
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@@
 <attribute name="VALUE" x="17.9705" y="39.743" size="0.4064" layer="28" rot="MR180"/>
 </element>
-<element name="R29" library="sfe" package="0402-RES" value="10K" x="14.4" y="6" smashed="yes" rot="R90">
-<attribute name="NAME" x="13.7015" y="5.111" size="0.4064" layer="25" rot="R90"/>
-<attribute name="VALUE" x="15.543" y="4.9205" size="0.4064" layer="27" rot="R90"/>
+<element name="R29" library="sfe" package="0402-RES" value="10K" x="14.4" y="6.4" smashed="yes" rot="R90">
+<attribute name="NAME" x="13.7015" y="5.511" size="0.4064" layer="25" rot="R90"/>
+<attribute name="VALUE" x="15.543" y="5.3205" size="0.4064" layer="27" rot="R90"/>
 </element>
 <element name="R32" library="sfe" package="0402-RES" value="1.13K" x="16.4" y="7.2" smashed="yes" rot="R90">
@@
 <attribute name="VIN_MIN_V" value="4.3" x="17.2" y="4" size="1.778" layer="27" display="off"/>
 </element>
-<element name="C53" library="SparkFun-Capacitors" library_urn="urn:adsk.eagle:library:510" package="0603" package3d_urn="urn:adsk.eagle:package:37414/1" value="4.7uF" x="14.4" y="3.25" smashed="yes" rot="R90">
-<attribute name="NAME" x="13.7015" y="2.361" size="0.4064" layer="25" rot="R90"/>
-<attribute name="PROD_ID" value="CAP-08280" x="14.4" y="3.25" size="1.778" layer="27" rot="R90" display="off"/>
-<attribute name="VALUE" value="4.7uF" x="15.543" y="2.1705" size="0.4064" layer="27" rot="R90"/>
+<element name="C53" library="SparkFun-Capacitors" library_urn="urn:adsk.eagle:library:510" package="0603" package3d_urn="urn:adsk.eagle:package:37414/1" value="4.7uF" x="14.4" y="3.65" smashed="yes" rot="R90">
+<attribute name="NAME" x="13.7015" y="2.761" size="0.4064" layer="25" rot="R90"/>
+<attribute name="PROD_ID" value="CAP-08280" x="14.4" y="3.65" size="1.778" layer="27" rot="R90" display="off"/>
+<attribute name="VALUE" value="4.7uF" x="15.543" y="2.5705" size="0.4064" layer="27" rot="R90"/>
 </element>
 <element name="C4" library="SparkFun-Capacitors" library_urn="urn:adsk.eagle:library:510" package="0603" package3d_urn="urn:adsk.eagle:package:37414/1" value="4.7uF" x="20.05" y="6.3" smashed="yes" rot="R270">
@@
 <attribute name="PURCHASE-URL" value="https://pricing.snapeda.com/search/part/RSP-122811-01/?ref=eda" x="7.6" y="32.8" size="1.778" layer="28" rot="MR0" display="off"/>
 <attribute name="VALUE" x="9.8" y="29.8" size="0.8128" layer="28" rot="MR0" align="top-left"/>
+</element>
+<element name="R46" library="sfe" package="0402-RES" value="1.5K" x="17.2" y="1.2" smashed="yes" rot="MR0">
+<attribute name="NAME" x="18.089" y="1.8985" size="0.4064" layer="26" rot="MR0"/>
+<attribute name="VALUE" x="18.2795" y="0.057" size="0.4064" layer="28" rot="MR0"/>
+</element>
+<element name="D26" library="SparkFun-LED" library_urn="urn:adsk.eagle:library:529" package="LED-0603" package3d_urn="urn:adsk.eagle:package:39354/1" value="GREEN" x="16" y="1.2" smashed="yes">
+<attribute name="NAME" x="16" y="1.835" size="0.6096" layer="25" font="vector" ratio="20" align="bottom-center"/>
+<attribute name="PROD_ID" value="DIO-00821" x="16" y="1.2" size="1.778" layer="27" display="off"/>
+<attribute name="VALUE" x="16" y="0.565" size="0.6096" layer="27" font="vector" ratio="20" align="top-center"/>
+</element>
+<element name="JP3" library="SparkFun-Jumpers" library_urn="urn:adsk.eagle:library:528" package="SMT-JUMPER_2_NC_PASTE_SILK" package3d_urn="urn:adsk.eagle:package:39282/1" value="JUMPER-SMT_2_NC_PASTE_SILK" x="14" y="1.6" smashed="yes" rot="MR90">
+<attribute name="NAME" x="15.143" y="1.6" size="0.6096" layer="26" font="vector" ratio="20" rot="MR90" align="bottom-center"/>
+<attribute name="VALUE" x="20" y="2.857" size="0.6096" layer="28" font="vector" ratio="20" rot="MR0" align="top-center"/>
+</element>
+<element name="JP4" library="SparkFun-Jumpers" library_urn="urn:adsk.eagle:library:528" package="SMT-JUMPER_2_NC_PASTE_SILK" package3d_urn="urn:adsk.eagle:package:39282/1" value="JUMPER-SMT_2_NC_PASTE_SILK" x="14" y="4" smashed="yes" rot="MR270">
+<attribute name="NAME" x="12.857" y="4" size="0.6096" layer="26" font="vector" ratio="20" rot="MR270" align="bottom-center"/>
+<attribute name="VALUE" x="20" y="5.143" size="0.6096" layer="28" font="vector" ratio="20" rot="MR180" align="top-center"/>
 </element>
 </elements>
@@
 <wire x1="17.95" y1="2.6" x2="16.95" y2="2.6" width="0" layer="19" extent="1-1"/>
 <wire x1="15.8" y1="3.25" x2="16.95" y2="2.6" width="0" layer="19" extent="1-1"/>
-<wire x1="14.4" y1="2.4" x2="15.8" y2="3.25" width="0" layer="19" extent="1-1"/>
-<wire x1="14.4" y1="6.65" x2="16.4" y2="7.85" width="0" layer="19" extent="1-1"/>
+<wire x1="14.4" y1="2.8" x2="15.8" y2="3.25" width="0" layer="19" extent="1-1"/>
+<wire x1="14.4" y1="7.05" x2="16.4" y2="7.85" width="0" layer="19" extent="1-1"/>
 <wire x1="20.25" y1="1.2" x2="17.95" y2="2.6" width="0" layer="19" extent="1-16"/>
 <wire x1="20.65" y1="4" x2="20.25" y2="1.2" width="0" layer="19" extent="16-16"/>
@@
 <wire x1="28.525" y1="21.407" x2="27.6" y2="20.5" width="0" layer="19" extent="1-16"/>
 <wire x1="28.65" y1="19.75" x2="27.6" y2="20.5" width="0" layer="19" extent="1-16"/>
-<wire x1="10.94" y1="1.6" x2="14.4" y2="2.4" width="0" layer="19" extent="1-1"/>
+<wire x1="10.94" y1="1.6" x2="14.4" y2="2.8" width="0" layer="19" extent="1-1"/>
 <wire x1="5.612" y1="16.587" x2="9.204" y2="16.1" width="0" layer="19" extent="1-16"/>
 <wire x1="3.8" y1="15.6" x2="5.612" y2="16.587" width="0" layer="19" extent="1-16"/>
@@
 <wire x1="3.8" y1="5.6" x2="3.8" y2="8" width="0" layer="19" extent="16-16"/>
 <wire x1="3.8" y1="3.2" x2="3.8" y2="5.6" width="0" layer="19" extent="16-16"/>
-<wire x1="10.652" y1="6.35" x2="14.4" y2="6.65" width="0" layer="19" extent="1-1"/>
+<wire x1="10.652" y1="6.35" x2="14.4" y2="7.05" width="0" layer="19" extent="1-1"/>
 <wire x1="9.8" y1="7.6" x2="10.652" y2="6.35" width="0" layer="19" extent="1-1"/>
 <wire x1="13.154" y1="34.756" x2="13.8" y2="30.25" width="0" layer="19" extent="16-16"/>
@@
 <contactref element="R29" pad="1"/>
 <contactref element="U11" pad="1"/>
-<wire x1="15.8" y1="4.75" x2="14.4" y2="5.35" width="0" layer="19" extent="1-1"/>
+<wire x1="15.8" y1="4.75" x2="14.4" y2="5.75" width="0" layer="19" extent="1-1"/>
 </signal>
 <signal name="ISET">
@@
 <contactref element="C53" pad="2"/>
 <contactref element="D21" pad="1"/>
-<wire x1="14.4" y1="4.1" x2="9.4" y2="7.6" width="0" layer="19" extent="1-1"/>
-<wire x1="15.8" y1="4.25" x2="14.4" y2="4.1" width="0" layer="19" extent="1-1"/>
+<wire x1="14.4" y1="4.5" x2="9.4" y2="7.6" width="0" layer="19" extent="1-1"/>
+<wire x1="15.8" y1="4.25" x2="14.4" y2="4.5" width="0" layer="19" extent="1-1"/>
 <wire x1="15.8" y1="3.75" x2="15.8" y2="4.25" width="0" layer="19" extent="1-1"/>
 <wire x1="8.652" y1="6.35" x2="9.4" y2="7.6" width="0" layer="19" extent="1-1"/>
@@
 <contactref element="U11" pad="10"/>
 <contactref element="C4" pad="2"/>
-<contactref element="R33" pad="2"/>
 <contactref element="U11" pad="5"/>
+<contactref element="JP3" pad="2"/>
+<contactref element="JP4" pad="2"/>
 <wire x1="20.05" y1="5.45" x2="25.7" y2="4.8" width="0" layer="19" extent="1-16"/>
-<wire x1="20" y1="3.85" x2="20.05" y2="5.45" width="0" layer="19" extent="1-1"/>
-<wire x1="18.6" y1="3.75" x2="20" y2="3.85" width="0" layer="19" extent="1-1"/>
-<wire x1="18.6" y1="4.25" x2="18.6" y2="3.75" width="0" layer="19" extent="1-1"/>
+<wire x1="18.6" y1="4.25" x2="20.05" y2="5.45" width="0" layer="19" extent="1-1"/>
+<wire x1="18.6" y1="3.75" x2="18.6" y2="4.25" width="0" layer="19" extent="1-1"/>
 <wire x1="16.45" y1="2.6" x2="18.6" y2="3.75" width="0" layer="19" extent="1-1"/>
+<wire x1="14" y1="2.0064" x2="16.45" y2="2.6" width="0" layer="19" extent="1-16"/>
+<wire x1="14" y1="3.5936" x2="14" y2="2.0064" width="0" layer="19" extent="16-16"/>
 </signal>
 <signal name="LED_B_INT">
@@
 <wire x1="18.323" y1="1.2" x2="20" y2="2.55" width="0" layer="19" extent="1-1"/>
 </signal>
+<signal name="N$1">
+<contactref element="D26" pad="A"/>
+<contactref element="R46" pad="1"/>
+<wire x1="15.123" y1="1.2" x2="17.85" y2="1.2" width="0" layer="19" extent="1-16"/>
+</signal>
+<signal name="N$9">
+<contactref element="D26" pad="C"/>
+<contactref element="U11" pad="7"/>
+<wire x1="16.877" y1="1.2" x2="17.45" y2="2.6" width="0" layer="19" extent="1-1"/>
+</signal>
+<signal name="N$11">
+<contactref element="R33" pad="2"/>
+<contactref element="JP4" pad="1"/>
+<wire x1="14" y1="4.4064" x2="20" y2="3.85" width="0" layer="19" extent="1-16"/>
+</signal>
+<signal name="N$12">
+<contactref element="R46" pad="2"/>
+<contactref element="JP3" pad="1"/>
+<wire x1="16.55" y1="1.2" x2="14" y2="1.1936" width="0" layer="19" extent="16-16"/>
+</signal>
 </signals>
