File: openmv5/rt10/rt10.sch (EAGLE design)
At the start: 216 parts, among them CN1 S2B-PH-K-S(LF)(SN), IC1 LM66200DRLR, IC2 AP61300Z6-7, IC3 IS42S16160G-6BL, IC4 ATECC608B-MAHDA-T, IC5 IS25LP064D-JKLE-TR, IC6 IS25LP128F-JKLE-TR, IC7 MXC4005XC, IC8 MIMXRT1052DVL6B, IC9 KSZ8081RNDCA-TR, J1 USB4105-GF-A, J2 DNP, J3 DNP, J4 DF12-36-DS, J5 USD-1040310811, J6 DNP, J7 DNP, J8 3221-10-0300-00, M1 9774030151R, M2 9774030151R, Q1 2N7002KW_R1_00001, Q2 2N7002KW_R1_00001, Q3 2N7002KW_R1_00001, Q4 2N7002KW_R1_00001, Q5 2N7002KW_R1_00001, U1 MIC5365-3.3YMT-TZ, U2 BQ24075RGTR, U3 LBEE5KL1DX-883, Y1 SC32S-7PF20PPM, Y2 XRCGB24M000F3M00R0

Commit message: Fix reverse protection on VIN, add TVS on FSIN, and fix USB current limits
Parts:
- added D11: CPDQT5V0HE-HF, CPDQT5V0HE-HF:CPDQT5V0HE-HF
- added Q6: PMXB120EPEZ, PMXB120EPEZ:PMXB120EPEZ
- R10: value 1.18K -> 3.3K; MPN AC0402FR-071K18L -> 0402WGJ0332TCE
- R12: value 1.13K -> 8.2K; MPN CRCW04021K13FKED -> RC0402JR-078K2L
Connections:
- new net VIN_INT: C5.2, IC1.VIN2, Q6.S
- net DCMI_FSIN: now also D11.1
- net GND: now also D11.2, Q6.G
- net VIN: now also Q6.D; no longer C5.2, IC1.VIN2
Changed lines of the file:
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@@
 <attribute name="MPN" value="UHD1110-FKA-CL1A13r3q1BBQFMF3"/>
 </part>
-<part name="R12" library="sfe" deviceset="RESISTOR" device="0402-RES" value="1.13K">
-<attribute name="MPN" value="CRCW04021K13FKED"/>
+<part name="R12" library="sfe" deviceset="RESISTOR" device="0402-RES" value="8.2K">
+<attribute name="MPN" value="RC0402JR-078K2L"/>
 </part>
 <part name="R11" library="sfe" deviceset="RESISTOR" device="0402-RES" value="46.4K">
 <attribute name="MPN" value="WR04X4642FTL"/>
 </part>
-<part name="R10" library="sfe" deviceset="RESISTOR" device="0402-RES" value="1.18K">
-<attribute name="MPN" value="AC0402FR-071K18L"/>
+<part name="R10" library="sfe" deviceset="RESISTOR" device="0402-RES" value="3.3K">
+<attribute name="MPN" value="0402WGJ0332TCE"/>
 </part>
 <part name="R9" library="sfe" deviceset="RESISTOR" device="0402-RES" value="10K">
@@
 <part name="FD4" library="SparkFun-Aesthetics" library_urn="urn:adsk.eagle:library:507" deviceset="FIDUCIAL" device="1X2" package3d_urn="urn:adsk.eagle:package:37108/1"/>
 <part name="FD8" library="SparkFun-Aesthetics" library_urn="urn:adsk.eagle:library:507" deviceset="FIDUCIAL" device="1X2" package3d_urn="urn:adsk.eagle:package:37108/1"/>
+<part name="Q6" library="PMXB120EPEZ" deviceset="PMXB120EPEZ" device="">
+<attribute name="MPN" value="PMXB120EPEZ"/>
+</part>
+<part name="D11" library="CPDQT5V0HE-HF" deviceset="CPDQT5V0HE-HF" device="">
+<attribute name="MPN" value="CPDQT5V0HE-HF"/>
+</part>
+<part name="GND36" library="SparkFun" deviceset="GND" device=""/>
 </parts>
 <sheets>
@@
 <attribute name="MPN" x="530.86" y="487.68" size="1.778" layer="96" rot="R180" display="off"/>
 </instance>
-<instance part="VIN2" gate="G$1" x="530.86" y="523.24" smashed="yes">
-<attribute name="VALUE" x="528.32" y="520.7" size="1.778" layer="96" rot="R90"/>
+<instance part="VIN2" gate="G$1" x="530.86" y="543.56" smashed="yes">
+<attribute name="VALUE" x="528.32" y="541.02" size="1.778" layer="96" rot="R90"/>
 </instance>
 <instance part="C4" gate="G$1" x="520.7" y="487.68" smashed="yes" rot="R180">
@@
 <attribute name="MPN" x="233.68" y="477.52" size="1.778" layer="96" rot="MR270" display="off"/>
 </instance>
-<instance part="RAW4" gate="G$1" x="520.7" y="523.24" smashed="yes">
-<attribute name="VALUE" x="518.16" y="520.7" size="1.778" layer="96" rot="R90"/>
+<instance part="RAW4" gate="G$1" x="520.7" y="543.56" smashed="yes">
+<attribute name="VALUE" x="518.16" y="541.02" size="1.778" layer="96" rot="R90"/>
 </instance>
 <instance part="RAW5" gate="G$1" x="614.68" y="523.24" smashed="yes">
@@
 <instance part="FD4" gate="G$1" x="833.12" y="330.2" smashed="yes"/>
 <instance part="FD8" gate="G$1" x="833.12" y="314.96" smashed="yes"/>
+<instance part="Q6" gate="G$1" x="538.48" y="525.78" smashed="yes" rot="MR0">
+<attribute name="NAME" x="527.05" y="529.59" size="1.778" layer="95" rot="MR0" align="center-left"/>
+<attribute name="VALUE" x="527.05" y="527.05" size="1.778" layer="96" rot="MR0" align="center-left"/>
+<attribute name="MPN" x="538.48" y="525.78" size="1.778" layer="96" rot="MR0" display="off"/>
+</instance>
+<instance part="D11" gate="G$1" x="553.72" y="203.2" smashed="yes" rot="R270">
+<attribute name="NAME" x="560.07" y="200.66" size="1.778" layer="95" rot="R270"/>
+<attribute name="VALUE" x="557.53" y="200.66" size="1.778" layer="96" rot="R270"/>
+<attribute name="MPN" x="553.72" y="203.2" size="1.778" layer="96" rot="R270" display="off"/>
+</instance>
+<instance part="GND36" gate="1" x="553.72" y="180.34" smashed="yes" rot="MR0">
+<attribute name="VALUE" x="556.26" y="177.8" size="1.778" layer="96" rot="MR0"/>
+</instance>
 </instances>
 <busses>
@@
 <wire x1="434.34" y1="472.44" x2="457.2" y2="472.44" width="0.1524" layer="91"/>
 <junction x="457.2" y="472.44"/>
+<pinref part="Q6" gate="G$1" pin="G"/>
+<wire x1="538.48" y1="525.78" x2="543.56" y2="525.78" width="0.1524" layer="91"/>
+<wire x1="543.56" y1="525.78" x2="543.56" y2="472.44" width="0.1524" layer="91"/>
+<wire x1="543.56" y1="472.44" x2="530.86" y2="472.44" width="0.1524" layer="91"/>
+<junction x="530.86" y="472.44"/>
 </segment>
 <segment>
@@
 <pinref part="GND35" gate="1" pin="GND"/>
 </segment>
+<segment>
+<pinref part="D11" gate="G$1" pin="2"/>
+<pinref part="GND36" gate="1" pin="GND"/>
+<wire x1="553.72" y1="193.04" x2="553.72" y2="182.88" width="0.1524" layer="91"/>
+</segment>
 </net>
 <net name="VBUS" class="0">
@@
 <wire x1="520.7" y1="513.08" x2="551.18" y2="513.08" width="0.1524" layer="91"/>
 <junction x="520.7" y="513.08"/>
-<wire x1="520.7" y1="513.08" x2="520.7" y2="523.24" width="0.1524" layer="91"/>
+<wire x1="520.7" y1="513.08" x2="520.7" y2="543.56" width="0.1524" layer="91"/>
 <pinref part="RAW4" gate="G$1" pin="RAW"/>
 </segment>
@@
 <net name="VIN" class="1">
 <segment>
-<pinref part="IC1" gate="G$1" pin="VIN2"/>
-<wire x1="500.38" y1="500.38" x2="530.86" y2="500.38" width="0.1524" layer="91"/>
-<pinref part="C5" gate="G$1" pin="2"/>
-<wire x1="530.86" y1="500.38" x2="530.86" y2="490.22" width="0.1524" layer="91"/>
-<pinref part="VIN2" gate="G$1" pin="VIN"/>
-<wire x1="530.86" y1="500.38" x2="530.86" y2="523.24" width="0.1524" layer="91"/>
-<junction x="530.86" y="500.38"/>
-</segment>
-<segment>
 <wire x1="802.64" y1="198.12" x2="792.48" y2="198.12" width="0.1524" layer="91"/>
 <wire x1="792.48" y1="198.12" x2="792.48" y2="220.98" width="0.1524" layer="91"/>
@@
 <junction x="792.48" y="220.98"/>
 </segment>
+<segment>
+<pinref part="Q6" gate="G$1" pin="D"/>
+<pinref part="VIN2" gate="G$1" pin="VIN"/>
+<wire x1="530.86" y1="535.94" x2="530.86" y2="543.56" width="0.1524" layer="91"/>
+</segment>
 </net>
 <net name="VDDA" class="0">
@@
 <pinref part="J4" gate="G$1" pin="23"/>
 <pinref part="R28" gate="G$1" pin="1"/>
-<wire x1="576.58" y1="223.52" x2="551.18" y2="223.52" width="0.1524" layer="91"/>
+<wire x1="576.58" y1="223.52" x2="553.72" y2="223.52" width="0.1524" layer="91"/>
 <label x="556.26" y="223.52" size="1.778" layer="95"/>
+<pinref part="D11" gate="G$1" pin="1"/>
+<wire x1="553.72" y1="223.52" x2="551.18" y2="223.52" width="0.1524" layer="91"/>
+<wire x1="553.72" y1="223.52" x2="553.72" y2="203.2" width="0.1524" layer="91"/>
+<junction x="553.72" y="223.52"/>
 </segment>
 <segment>
@@
 </segment>
 </net>
+<net name="VIN_INT" class="1">
+<segment>
+<pinref part="IC1" gate="G$1" pin="VIN2"/>
+<wire x1="500.38" y1="500.38" x2="530.86" y2="500.38" width="0.1524" layer="91"/>
+<pinref part="C5" gate="G$1" pin="2"/>
+<wire x1="530.86" y1="500.38" x2="530.86" y2="490.22" width="0.1524" layer="91"/>
+<pinref part="Q6" gate="G$1" pin="S"/>
+<wire x1="530.86" y1="520.7" x2="530.86" y2="500.38" width="0.1524" layer="91"/>
+<junction x="530.86" y="500.38"/>
+</segment>
+</net>

Commit message: Final
Parts:
- removed D11: CPDQT5V0HE-HF, CPDQT5V0HE-HF:CPDQT5V0HE-HF
- removed L3: 100, sfe:INDUCTOR0402
- added C110: 1nF, sfe:CAP0402-CAP
- added R41: 1M, sfe:RESISTOR0402-RES
Connections:
- net DCMI_FSIN: no longer D11.1
- net GND: now also C110.1, R41.2; no longer D11.2, L3.1
- net SHELL_GND: now also C110.2, R41.1; no longer L3.2
Changed lines of the file:
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@@
 <attribute name="MPN" value="LBEE5KL1DX-883"/>
 </part>
-<part name="L3" library="sfe" deviceset="INDUCTOR" device="0402" value="100">
-<attribute name="MPN" value="MFBM1V1608-101-R"/>
-</part>
 <part name="VBUS3" library="supply" deviceset="VBUS" device=""/>
 <part name="J2" library="SparkFun-Connectors" library_urn="urn:adsk.eagle:library:513" deviceset="CONN_08" device="&quot;" package3d_urn="urn:adsk.eagle:package:38138/1" value="DNP">
@@
 <attribute name="MPN" value="PMXB120EPEZ"/>
 </part>
-<part name="D11" library="CPDQT5V0HE-HF" deviceset="CPDQT5V0HE-HF" device="">
-<attribute name="MPN" value="CPDQT5V0HE-HF"/>
+<part name="R41" library="sfe" deviceset="RESISTOR" device="0402-RES" value="1M">
+<attribute name="MPN" value="0402WGF1004TCE"/>
+</part>
+<part name="C110" library="sfe" deviceset="CAP" device="0402-CAP" value="1nF">
+<attribute name="MPN" value="C0402C102K5RAC"/>
 </part>
-<part name="GND36" library="SparkFun" deviceset="GND" device=""/>
 </parts>
 <sheets>
@@
 <attribute name="VALUE" x="713.73" y="50.28" size="2.540909375" layer="96"/>
 </instance>
-<instance part="L3" gate="G$1" x="96.52" y="492.76" smashed="yes" rot="R270">
-<attribute name="NAME" x="101.6" y="490.22" size="1.778" layer="95" font="vector" rot="R270"/>
-<attribute name="VALUE" x="91.44" y="490.22" size="1.778" layer="96" font="vector" rot="R270"/>
-<attribute name="MPN" x="96.52" y="492.76" size="1.778" layer="96" rot="R270" display="off"/>
-</instance>
 <instance part="VBUS3" gate="G$1" x="132.08" y="523.24" smashed="yes">
 <attribute name="VALUE" x="129.54" y="520.7" size="1.778" layer="96" rot="R90"/>
@@
 <attribute name="MPN" x="538.48" y="525.78" size="1.778" layer="96" rot="MR0" display="off"/>
 </instance>
-<instance part="D11" gate="G$1" x="553.72" y="203.2" smashed="yes" rot="R270">
-<attribute name="NAME" x="560.07" y="200.66" size="1.778" layer="95" rot="R270"/>
-<attribute name="VALUE" x="557.53" y="200.66" size="1.778" layer="96" rot="R270"/>
-<attribute name="MPN" x="553.72" y="203.2" size="1.778" layer="96" rot="R270" display="off"/>
-</instance>
-<instance part="GND36" gate="1" x="553.72" y="180.34" smashed="yes" rot="MR0">
-<attribute name="VALUE" x="556.26" y="177.8" size="1.778" layer="96" rot="MR0"/>
+<instance part="R41" gate="G$1" x="88.9" y="485.14" smashed="yes" rot="R270">
+<attribute name="MPN" x="88.9" y="485.14" size="1.778" layer="96" rot="R270" display="off"/>
+<attribute name="NAME" x="90.3986" y="488.95" size="1.778" layer="95" rot="R270"/>
+<attribute name="VALUE" x="85.598" y="488.95" size="1.778" layer="96" rot="R270"/>
+</instance>
+<instance part="C110" gate="G$1" x="101.6" y="487.68" smashed="yes" rot="R180">
+<attribute name="NAME" x="100.076" y="484.759" size="1.778" layer="95" rot="MR270"/>
+<attribute name="VALUE" x="100.076" y="489.839" size="1.778" layer="96" rot="R90"/>
+<attribute name="MPN" x="101.6" y="487.68" size="1.778" layer="96" rot="R180" display="off"/>
 </instance>
 </instances>
@@
 <wire x1="180.34" y1="500.38" x2="180.34" y2="477.52" width="0.1524" layer="91"/>
 <junction x="180.34" y="500.38"/>
-<wire x1="27.94" y1="477.52" x2="111.76" y2="477.52" width="0.1524" layer="91"/>
-<pinref part="L3" gate="G$1" pin="1"/>
+<wire x1="27.94" y1="477.52" x2="88.9" y2="477.52" width="0.1524" layer="91"/>
+<wire x1="88.9" y1="477.52" x2="101.6" y2="477.52" width="0.1524" layer="91"/>
+<wire x1="101.6" y1="477.52" x2="111.76" y2="477.52" width="0.1524" layer="91"/>
 <wire x1="111.76" y1="477.52" x2="121.92" y2="477.52" width="0.1524" layer="91"/>
 <wire x1="121.92" y1="477.52" x2="132.08" y2="477.52" width="0.1524" layer="91"/>
 <wire x1="132.08" y1="477.52" x2="180.34" y2="477.52" width="0.1524" layer="91"/>
-<wire x1="101.6" y1="492.76" x2="111.76" y2="492.76" width="0.1524" layer="91"/>
-<wire x1="111.76" y1="492.76" x2="111.76" y2="477.52" width="0.1524" layer="91"/>
+<wire x1="111.76" y1="495.3" x2="111.76" y2="477.52" width="0.1524" layer="91"/>
 <pinref part="J1" gate="G$1" pin="GND"/>
 <wire x1="78.74" y1="495.3" x2="111.76" y2="495.3" width="0.1524" layer="91"/>
-<wire x1="111.76" y1="495.3" x2="111.76" y2="492.76" width="0.1524" layer="91"/>
-<junction x="111.76" y="492.76"/>
 <junction x="111.76" y="477.52"/>
 <pinref part="R7" gate="G$1" pin="2"/>
@@
 <pinref part="FL1" gate="G$1" pin="GND_2"/>
 <pinref part="FL1" gate="G$1" pin="GND_1"/>
+<pinref part="R41" gate="G$1" pin="2"/>
+<wire x1="88.9" y1="480.06" x2="88.9" y2="477.52" width="0.1524" layer="91"/>
+<junction x="88.9" y="477.52"/>
+<pinref part="C110" gate="G$1" pin="1"/>
+<wire x1="101.6" y1="482.6" x2="101.6" y2="477.52" width="0.1524" layer="91"/>
+<junction x="101.6" y="477.52"/>
 </segment>
 <segment>
@@
 <pinref part="GND35" gate="1" pin="GND"/>
 </segment>
-<segment>
-<pinref part="D11" gate="G$1" pin="2"/>
-<pinref part="GND36" gate="1" pin="GND"/>
-<wire x1="553.72" y1="193.04" x2="553.72" y2="182.88" width="0.1524" layer="91"/>
-</segment>
 </net>
 <net name="VBUS" class="0">
@@
 <segment>
 <pinref part="J1" gate="G$1" pin="SHELL_GND"/>
-<pinref part="L3" gate="G$1" pin="2"/>
 <wire x1="78.74" y1="492.76" x2="88.9" y2="492.76" width="0.1524" layer="91"/>
+<pinref part="R41" gate="G$1" pin="1"/>
+<wire x1="88.9" y1="492.76" x2="88.9" y2="490.22" width="0.1524" layer="91"/>
+<wire x1="88.9" y1="492.76" x2="101.6" y2="492.76" width="0.1524" layer="91"/>
+<junction x="88.9" y="492.76"/>
+<pinref part="C110" gate="G$1" pin="2"/>
+<wire x1="101.6" y1="492.76" x2="101.6" y2="490.22" width="0.1524" layer="91"/>
 </segment>
 </net>
@@
 <pinref part="J4" gate="G$1" pin="23"/>
 <pinref part="R28" gate="G$1" pin="1"/>
-<wire x1="576.58" y1="223.52" x2="553.72" y2="223.52" width="0.1524" layer="91"/>
+<wire x1="576.58" y1="223.52" x2="551.18" y2="223.52" width="0.1524" layer="91"/>
 <label x="556.26" y="223.52" size="1.778" layer="95"/>
-<pinref part="D11" gate="G$1" pin="1"/>
-<wire x1="553.72" y1="223.52" x2="551.18" y2="223.52" width="0.1524" layer="91"/>
-<wire x1="553.72" y1="223.52" x2="553.72" y2="203.2" width="0.1524" layer="91"/>
-<junction x="553.72" y="223.52"/>
 </segment>
 <segment>

Commit message: Fix issues with part selection
Parts:
- L1: device sfe:INDUCTOR0402 -> SparkFun-Coils:INDUCTOR-0603-33NH
- L4, L6, L8: MPN MFBM1V1608-101-R -> MFBM1V1005-101-R
- R6, R7: MPN RMC1/20-512FPA -> RC0402JR-075K1L
Changed lines of the file:
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@@
 </part>
 <part name="R6" library="sfe" deviceset="RESISTOR" device="0402-RES" value="5.1K">
-<attribute name="MPN" value="RMC1/20-512FPA"/>
+<attribute name="MPN" value="RC0402JR-075K1L"/>
 </part>
 <part name="R7" library="sfe" deviceset="RESISTOR" device="0402-RES" value="5.1K">
-<attribute name="MPN" value="RMC1/20-512FPA"/>
-</part>
-<part name="L1" library="sfe" deviceset="INDUCTOR" device="0402" value="100">
-<attribute name="MPN" value="MFBM1V1608-101-R"/>
+<attribute name="MPN" value="RC0402JR-075K1L"/>
 </part>
 <part name="GND19" library="sfe" deviceset="GND" device=""/>
@@
 </part>
 <part name="L4" library="sfe" deviceset="INDUCTOR" device="0402" value="100">
-<attribute name="MPN" value="MFBM1V1608-101-R"/>
+<attribute name="MPN" value="MFBM1V1005-101-R"/>
 </part>
 <part name="C51" library="SparkFun-Capacitors" library_urn="urn:adsk.eagle:library:510" deviceset="22UF" device="-0805-6.3V-20%" package3d_urn="urn:adsk.eagle:package:37429/1" value="22uF">
@@
 </part>
 <part name="L8" library="sfe" deviceset="INDUCTOR" device="0402" value="100">
-<attribute name="MPN" value="MFBM1V1608-101-R"/>
+<attribute name="MPN" value="MFBM1V1005-101-R"/>
 </part>
 <part name="P+10" library="SparkFun" deviceset="VCC" device=""/>
@@
 </part>
 <part name="L6" library="sfe" deviceset="INDUCTOR" device="0402" value="100">
-<attribute name="MPN" value="MFBM1V1608-101-R"/>
+<attribute name="MPN" value="MFBM1V1005-101-R"/>
 </part>
 <part name="C60" library="sfe" deviceset="CAP" device="0402-CAP" value="4.7uF">
@@
 <attribute name="MPN" value="C0402C102K5RAC"/>
 </part>
+<part name="L1" library="SparkFun-Coils" library_urn="urn:adsk.eagle:library:512" deviceset="INDUCTOR" device="-0603-33NH" package3d_urn="urn:adsk.eagle:package:37574/1" value="100">
+<attribute name="MPN" value="MFBM1V1608-101-R"/>
+</part>
 </parts>
 <sheets>
@@
 <attribute name="VALUE" x="118.618" y="496.57" size="1.778" layer="96" rot="R270"/>
 </instance>
-<instance part="L1" gate="G$1" x="93.98" y="513.08" smashed="yes" rot="R90">
-<attribute name="NAME" x="88.9" y="515.62" size="1.778" layer="95" font="vector" rot="R90"/>
-<attribute name="VALUE" x="99.06" y="515.62" size="1.778" layer="96" font="vector" rot="R90"/>
-<attribute name="MPN" x="93.98" y="513.08" size="1.778" layer="96" rot="R90" display="off"/>
-</instance>
 <instance part="GND19" gate="1" x="132.08" y="464.82" smashed="yes" rot="MR0">
 <attribute name="VALUE" x="134.62" y="462.28" size="1.778" layer="96" rot="MR0"/>
@@
 <attribute name="MPN" x="101.6" y="487.68" size="1.778" layer="96" rot="R180" display="off"/>
 </instance>
+<instance part="L1" gate="G$1" x="93.98" y="513.08" smashed="yes" rot="R90">
+<attribute name="NAME" x="91.44" y="514.35" size="1.778" layer="95" font="vector" rot="R90"/>
+<attribute name="VALUE" x="96.52" y="514.35" size="1.778" layer="96" font="vector" rot="R90" align="top-left"/>
+<attribute name="MPN" x="93.98" y="513.08" size="1.778" layer="96" rot="R90" display="off"/>
+</instance>
 </instances>
 <busses>
@@
 <wire x1="137.16" y1="508" x2="132.08" y2="508" width="0.1524" layer="91"/>
 <wire x1="132.08" y1="508" x2="132.08" y2="513.08" width="0.1524" layer="91"/>
-<pinref part="L1" gate="G$1" pin="2"/>
-<wire x1="132.08" y1="513.08" x2="101.6" y2="513.08" width="0.1524" layer="91"/>
+<wire x1="132.08" y1="513.08" x2="99.06" y2="513.08" width="0.1524" layer="91"/>
 <pinref part="VBUS3" gate="G$1" pin="VBUS"/>
 <wire x1="132.08" y1="523.24" x2="132.08" y2="513.08" width="0.1524" layer="91"/>
 <junction x="132.08" y="513.08"/>
 <pinref part="FL1" gate="G$1" pin="VBUS"/>
+<pinref part="L1" gate="G$1" pin="2"/>
 </segment>
 <segment>
@@
 <net name="USB_VBUS" class="0">
 <segment>
-<pinref part="L1" gate="G$1" pin="1"/>
 <pinref part="J1" gate="G$1" pin="VBUS"/>
 <wire x1="78.74" y1="513.08" x2="83.82" y2="513.08" width="0.1524" layer="91"/>
@@
 <junction x="83.82" y="513.08"/>
 <pinref part="FL1" gate="G$1" pin="ID"/>
+<pinref part="L1" gate="G$1" pin="1"/>
 </segment>
 </net>

Commit message: Update remaining MPNs
Parts:
- C110: MPN C0402C102K5RAC -> VJ0402Y102JXACW1BC
- R10: MPN 0402WGJ0332TCE -> CRCW04023K30FKEDC
- R33, R37, R9: MPN AC0402FR-1310KL -> CRCW04021K00FKEDC
- R41: MPN 0402WGF1004TCE -> CRCW04021M00FKEDC
Changed lines of the file:
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@@
 </part>
 <part name="R10" library="sfe" deviceset="RESISTOR" device="0402-RES" value="3.3K">
-<attribute name="MPN" value="0402WGJ0332TCE"/>
+<attribute name="MPN" value="CRCW04023K30FKEDC"/>
 </part>
 <part name="R9" library="sfe" deviceset="RESISTOR" device="0402-RES" value="10K">
-<attribute name="MPN" value="AC0402FR-1310KL"/>
+<attribute name="MPN" value="CRCW04021K00FKEDC"/>
 </part>
 <part name="C9" library="sfe" deviceset="CAP" device="0402-CAP" value="4.7uF">
@@
 <part name="GND1" library="sfe" deviceset="GND" device=""/>
 <part name="R37" library="sfe" deviceset="RESISTOR" device="0402-RES" value="10K">
-<attribute name="MPN" value="AC0402FR-1310KL"/>
+<attribute name="MPN" value="CRCW04021K00FKEDC"/>
 </part>
 <part name="R29" library="sfe" deviceset="RESISTOR" device="0402-RES" value="100K">
@@
 </part>
 <part name="R33" library="sfe" deviceset="RESISTOR" device="0402-RES" value="10K">
-<attribute name="MPN" value="AC0402FR-1310KL"/>
+<attribute name="MPN" value="CRCW04021K00FKEDC"/>
 </part>
 <part name="C21" library="sfe" deviceset="CAP" device="0402-CAP" value="4.7uF">
@@
 </part>
 <part name="R41" library="sfe" deviceset="RESISTOR" device="0402-RES" value="1M">
-<attribute name="MPN" value="0402WGF1004TCE"/>
+<attribute name="MPN" value="CRCW04021M00FKEDC"/>
 </part>
 <part name="C110" library="sfe" deviceset="CAP" device="0402-CAP" value="1nF">
-<attribute name="MPN" value="C0402C102K5RAC"/>
+<attribute name="MPN" value="VJ0402Y102JXACW1BC"/>
 </part>
 <part name="L1" library="SparkFun-Coils" library_urn="urn:adsk.eagle:library:512" deviceset="INDUCTOR" device="-0603-33NH" package3d_urn="urn:adsk.eagle:package:37574/1" value="100">

Commit message: Try again
Parts:
- R1, R26, R36, R39, R4, R5: MPN 0402WGF1001TCE -> CRCW04021K00FKEDC
- R33, R37, R9: MPN CRCW04021K00FKEDC -> AC0402FR-1310KL
Changed lines of the file:
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@@
 </part>
 <part name="R9" library="sfe" deviceset="RESISTOR" device="0402-RES" value="10K">
-<attribute name="MPN" value="CRCW04021K00FKEDC"/>
+<attribute name="MPN" value="AC0402FR-1310KL"/>
 </part>
 <part name="C9" library="sfe" deviceset="CAP" device="0402-CAP" value="4.7uF">
@@
 </part>
 <part name="R1" library="sfe" deviceset="RESISTOR" device="0402-RES" value="1K">
-<attribute name="MPN" value="0402WGF1001TCE"/>
+<attribute name="MPN" value="CRCW04021K00FKEDC"/>
 </part>
 <part name="R4" library="sfe" deviceset="RESISTOR" device="0402-RES" value="1K">
-<attribute name="MPN" value="0402WGF1001TCE"/>
+<attribute name="MPN" value="CRCW04021K00FKEDC"/>
 </part>
 <part name="IC1" library="LM66200DRLR" deviceset="LM66200DRLR" device="">
@@
 </part>
 <part name="R5" library="sfe" deviceset="RESISTOR" device="0402-RES" value="1K">
-<attribute name="MPN" value="0402WGF1001TCE"/>
+<attribute name="MPN" value="CRCW04021K00FKEDC"/>
 </part>
 <part name="C2" library="sfe" deviceset="CAP" device="0402-CAP" value="4.7uF">
@@
 <part name="GND1" library="sfe" deviceset="GND" device=""/>
 <part name="R37" library="sfe" deviceset="RESISTOR" device="0402-RES" value="10K">
-<attribute name="MPN" value="CRCW04021K00FKEDC"/>
+<attribute name="MPN" value="AC0402FR-1310KL"/>
 </part>
 <part name="R29" library="sfe" deviceset="RESISTOR" device="0402-RES" value="100K">
@@
 <part name="P+10" library="SparkFun" deviceset="VCC" device=""/>
 <part name="R36" library="sfe" deviceset="RESISTOR" device="0402-RES" value="1K">
-<attribute name="MPN" value="0402WGF1001TCE"/>
+<attribute name="MPN" value="CRCW04021K00FKEDC"/>
 </part>
 <part name="P+11" library="SparkFun" deviceset="VCC" device=""/>
 <part name="R39" library="sfe" deviceset="RESISTOR" device="0402-RES" value="1K">
-<attribute name="MPN" value="0402WGF1001TCE"/>
+<attribute name="MPN" value="CRCW04021K00FKEDC"/>
 </part>
 <part name="FL2" library="EMIF06-1005M12" deviceset="EMIF06-1005M12" device="">
@@
 </part>
 <part name="R33" library="sfe" deviceset="RESISTOR" device="0402-RES" value="10K">
-<attribute name="MPN" value="CRCW04021K00FKEDC"/>
+<attribute name="MPN" value="AC0402FR-1310KL"/>
 </part>
 <part name="C21" library="sfe" deviceset="CAP" device="0402-CAP" value="4.7uF">
@@
 </part>
 <part name="R26" library="sfe" deviceset="RESISTOR" device="0402-RES" value="1K">
-<attribute name="MPN" value="0402WGF1001TCE"/>
+<attribute name="MPN" value="CRCW04021K00FKEDC"/>
 </part>
 <part name="U1" library="MIC5365-3.3YMT-TZ" deviceset="MIC5365-3.3YMT-TZ" device="">
