File: openmv5/rs422-rs485/rs422-rs485.brd (EAGLE design)
At the start: 35.6 x 26.7 mm, 94 parts, among them IC1 TPS613222ADBVR, IC2 AP64060WU-7, IC3 LM321LVIDCKR, IC4 74LVC1G07GW,125, IC5 THVD1426DR, IC6 THVD1426DR, J1 OPENMV5-TOP, J2 1771088, Q1 SSM3J356R,LF, U1 74LVC1G17SE-7, U2 74AHC1G08SE-7

Commit message: Fix labeling
Routing:
- net GND: track 225.4 -> 223.8 mm
- net RS422_RXI: track 19.6 -> 18.0 mm
- net RS422_TXO: track 19.5 -> 20.6 mm
Other:
- board text added: "A+"
- board text added: "AIN - 0 to 5V or 4-20mA"
- board text added: "B-"
- board text added: "PWR - 6V to 36V"
- board text added: "RS422 Y/Z/A/B"
- board text added: "SYN - 0 to 5V I/O"
- board text added: "YA+"
- board text added: "ZB-"
- board text removed: "A"
- board text removed: "AIN: 0-5V or 4-20mA"
- board text removed: "B"
- board text removed: "PWR: 6V to 36V"
- board text removed: "SYN: 0-5V I/O"
- board text removed: "Y/Z/A/B RS422"
- board text removed: "YA"
- board text removed: "ZB"
Changed lines of the file:
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@@
 <text x="24.3" y="12.6" size="0.8128" layer="21" font="vector" ratio="22">AIN</text>
 <text x="26.8" y="12.6" size="0.8128" layer="21" font="vector" ratio="22">SYN</text>
-<text x="14.7" y="12.6" size="0.8128" layer="21" font="vector" ratio="22">ZB</text>
-<text x="17.2" y="12.6" size="0.8128" layer="21" font="vector" ratio="22">YA</text>
-<text x="19.3" y="13.5" size="0.8128" layer="22" font="vector" ratio="22" rot="MR180">TRM</text>
-<text x="16.7" y="13.5" size="0.8128" layer="22" font="vector" ratio="22" rot="MR180">TRM</text>
-<text x="20" y="12.6" size="0.8128" layer="21" font="vector" ratio="22">B</text>
-<text x="22.4" y="12.6" size="0.8128" layer="21" font="vector" ratio="22">A</text>
+<text x="14.3" y="12.6" size="0.8128" layer="21" font="vector" ratio="22">ZB-</text>
+<text x="16.8" y="12.6" size="0.8128" layer="21" font="vector" ratio="22">YA+</text>
+<text x="19.2" y="13.5" size="0.8128" layer="22" font="vector" ratio="22" rot="MR180">TRM</text>
+<text x="16.6" y="13.5" size="0.8128" layer="22" font="vector" ratio="22" rot="MR180">TRM</text>
+<text x="19.7" y="12.6" size="0.8128" layer="21" font="vector" ratio="22">B-</text>
+<text x="22.2" y="12.6" size="0.8128" layer="21" font="vector" ratio="22">A+</text>
 <text x="32.4" y="5.3" size="0.8128" layer="22" font="vector" ratio="22" rot="MR270">VIN</text>
 <text x="10.5" y="26.3" size="0.8128" layer="21" font="vector" ratio="22" rot="R270">TXO
@@
 <text x="27.3" y="13" size="0.8128" layer="22" font="vector" ratio="22" rot="MR0">I</text>
 <text x="24.1" y="14.8" size="0.8128" layer="21" font="vector" ratio="22" rot="R90">mA</text>
-<text x="13.6" y="25.2" size="0.8128" layer="21" font="vector" ratio="20">PWR: 6V to 36V </text>
-<text x="13.6" y="24" size="0.8128" layer="21" font="vector" ratio="20">AIN: 0-5V or 4-20mA</text>
-<text x="13.6" y="22.8" size="0.8128" layer="21" font="vector" ratio="20">SYN: 0-5V I/O</text>
-<text x="21.8" y="13.5" size="0.8128" layer="22" font="vector" ratio="22" rot="MR180">TRM</text>
+<text x="13.6" y="25.2" size="0.8128" layer="21" font="vector" ratio="20">PWR - 6V to 36V </text>
+<text x="13.6" y="24" size="0.8128" layer="21" font="vector" ratio="20">AIN - 0 to 5V or 4-20mA</text>
+<text x="13.6" y="22.8" size="0.8128" layer="21" font="vector" ratio="20">SYN - 0 to 5V I/O</text>
+<text x="21.6" y="13.5" size="0.8128" layer="22" font="vector" ratio="22" rot="MR180">TRM</text>
 <text x="13.3" y="14" size="0.8128" layer="22" font="vector" ratio="22" rot="MR90">TRM</text>
-<text x="14.2" y="17.2" size="0.8128" layer="21" font="vector" ratio="22" rot="R90">RS485
+<text x="8.2" y="16.2" size="0.8128" layer="21" font="vector" ratio="22" rot="R90">RS485
 YA/ZB</text>
-<text x="25.7" y="18.5" size="0.8128" layer="21" font="vector" ratio="22" rot="R90">Y/Z/A/B
-  RS422</text>
+<text x="14.2" y="16.2" size="0.8128" layer="21" font="vector" ratio="22" rot="R90">RS422
+Y/Z/A/B</text>
 </plain>
 <attributes>
@@
 <via x="11" y="20.8" extent="1-16" drill="0.4064"/>
 <wire x1="11" y1="20.8" x2="11" y2="21.5" width="0.4064" layer="1"/>
-<via x="6" y="22.8" extent="1-16" drill="0.4064"/>
+<via x="6" y="22" extent="1-16" drill="0.4064"/>
 <via x="26" y="20.4" extent="1-16" drill="0.254"/>
 <wire x1="20.9" y1="11.2" x2="24.15" y2="11.2" width="0.254" layer="16"/>
@@
 <via x="23.5" y="12.5" extent="1-16" drill="0.254"/>
 <wire x1="8.3" y1="20.6" x2="8.85" y2="20.6" width="0.4064" layer="1"/>
-<wire x1="6.1" y1="21" x2="6.1" y2="22.7" width="0.4064" layer="1"/>
-<wire x1="6.1" y1="22.7" x2="6" y2="22.8" width="0.4064" layer="1"/>
-<wire x1="6" y1="22.8" x2="6" y2="18.4" width="0.4064" layer="16"/>
+<wire x1="6.1" y1="21" x2="6.1" y2="21.9" width="0.4064" layer="1"/>
+<wire x1="6.1" y1="21.9" x2="6" y2="22" width="0.4064" layer="1"/>
+<wire x1="6" y1="22" x2="6" y2="18.4" width="0.4064" layer="16"/>
 <wire x1="6" y1="18.4" x2="6" y2="16" width="0.4064" layer="16"/>
 <wire x1="6" y1="16" x2="8.84" y2="13.16" width="0.4064" layer="16"/>
@@
 <contactref element="D10" pad="1"/>
 <contactref element="IC5" pad="4"/>
-<via x="6.8" y="23.6" extent="1-16" drill="0.254"/>
-<wire x1="6.8" y1="23.6" x2="8.1" y2="24.9" width="0.254" layer="16"/>
-<wire x1="8.1" y1="24.9" x2="13.1" y2="24.9" width="0.254" layer="16"/>
+<via x="6.8" y="22" extent="1-16" drill="0.254"/>
+<wire x1="6.8" y1="22" x2="9.7" y2="24.9" width="0.254" layer="16"/>
+<wire x1="9.7" y1="24.9" x2="13.1" y2="24.9" width="0.254" layer="16"/>
 <via x="13.1" y="24.9" extent="1-16" drill="0.254"/>
 <wire x1="6.4" y1="15.45" x2="6.8" y2="15.85" width="0.254" layer="1"/>
-<wire x1="6.8" y1="23.6" x2="6.8" y2="20.2" width="0.254" layer="1"/>
-<wire x1="6.8" y1="20" x2="6.8" y2="15.85" width="0.254" layer="1"/>
-<wire x1="9.4064" y1="25.2" x2="9.4064" y2="25.6" width="0.254" layer="1"/>
-<wire x1="6.8" y1="23.6" x2="6.8" y2="20.8" width="0.254" layer="16"/>
+<wire x1="6.8" y1="22" x2="6.8" y2="20.2" width="0.254" layer="1"/>
+<wire x1="6.8" y1="20.2" x2="6.8" y2="15.85" width="0.254" layer="1"/>
+<wire x1="6.8" y1="22" x2="6.8" y2="20.8" width="0.254" layer="16"/>
 <wire x1="6.8" y1="20.8" x2="7.289" y2="20.8" width="0.254" layer="16"/>
 <wire x1="7.289" y1="20.8" x2="7.289" y2="20.805" width="0.254" layer="16"/>
 <wire x1="6.1" y1="20.2" x2="6.8" y2="20.2" width="0.254" layer="1"/>
-<wire x1="6.8" y1="20.2" x2="6.8" y2="20" width="0.254" layer="1"/>
-<wire x1="6.8" y1="23.6" x2="9.4064" y2="25.2" width="0" layer="19" extent="1-1"/>
+<wire x1="13.1" y1="24.9" x2="9.4064" y2="24.9" width="0.254" layer="1"/>
+<wire x1="9.4064" y1="24.9" x2="9.4064" y2="25.2" width="0.254" layer="1"/>
 </signal>
 <signal name="RS422_RXI" class="4">
@@
 <contactref element="U2" pad="4"/>
 <wire x1="7.7" y1="15.45" x2="7.4" y2="15.75" width="0.254" layer="1"/>
-<via x="7.4" y="23.2" extent="1-16" drill="0.254"/>
-<wire x1="7.4" y1="23.2" x2="8.2" y2="22.4" width="0.254" layer="16"/>
-<wire x1="13.1" y1="22.4" x2="8.2" y2="22.4" width="0.254" layer="16"/>
+<via x="7.4" y="21.6" extent="1-16" drill="0.254"/>
+<wire x1="7.4" y1="21.6" x2="8.19999375" y2="22.4" width="0.254" layer="16"/>
+<wire x1="13.1" y1="22.4" x2="8.19999375" y2="22.4" width="0.254" layer="16"/>
 <via x="13.1" y="22.4" extent="1-16" drill="0.254"/>
 <wire x1="7.4" y1="15.75" x2="7.4" y2="17.3" width="0.254" layer="1"/>
@@
 <wire x1="7.4" y1="17.3" x2="7.4" y2="20.5" width="0.254" layer="1"/>
 <wire x1="7.4" y1="20.5" x2="7.5" y2="20.6" width="0.254" layer="1"/>
-<wire x1="7.4" y1="23.2" x2="7.4" y2="20.5" width="0.254" layer="1"/>
+<wire x1="7.4" y1="21.6" x2="7.4" y2="20.5" width="0.254" layer="1"/>
 <wire x1="13.1" y1="22.4" x2="9.4064" y2="22.4" width="0.254" layer="1"/>
 <wire x1="9.4064" y1="22.4" x2="9.4064" y2="22.8" width="0.254" layer="1"/>
