File: openmv5/rs422-rs485/rs422-rs485.brd (EAGLE design)
At the start: 35.6 x 26.7 mm, 94 parts, among them IC1 TPS613222ADBVR, IC2 AP64060WU-7, IC3 LM321LVIDCKR, IC4 74LVC1G07GW,125, IC5 THVD1426DR, IC6 THVD1426DR, J1 OPENMV5-TOP, J2 1771088, Q1 SSM3J356R,LF, U1 74LVC1G17SE-7, U2 74AHC1G08SE-7

Commit message: Fix drc issues
Parts:
- moved FD3 0.41 mm to (6.90, 12.8)
- moved FD4 0.41 mm to (6.90, 12.8)
- moved JP3 0.40 mm to (6.60, 8.60)
- moved FD5 0.20 mm to (34.2, 21.6)
- moved FD1 0.14 mm to (29.5, 13.4)
- moved FD2 0.14 mm to (29.5, 13.4)
Routing:
- net YA: track 13.5 -> 14.3 mm

Commit message: Add servo shield
Other:
- board text added: "ADC P6"
- board text added: "FSYNC P10"
- board text removed: "ADC P11"
- board text removed: "FSYNC P11"
Changed lines of the file:
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@@
 <text x="32.4" y="2.8" size="0.8128" layer="22" font="vector" ratio="22" rot="MR270">GND</text>
 <text x="28.8" y="17.5" size="0.8128" layer="22" font="vector" ratio="22" rot="MR180">FSYNC
-P11</text>
+P10</text>
 <text x="11.9" y="12.6" size="0.8128" layer="21" font="vector" ratio="22">GND</text>
 <text x="9.4" y="12.6" size="0.8128" layer="21" font="vector" ratio="22">PWR</text>
@@
 P5</text>
 <text x="5.6" y="9.9" size="0.8128" layer="22" font="vector" ratio="22" rot="MR90">ADC
-P11</text>
+P6</text>
 <text x="28.9" y="13" size="0.8128" layer="22" font="vector" ratio="22" rot="MR0">O</text>
 <text x="27.3" y="13" size="0.8128" layer="22" font="vector" ratio="22" rot="MR0">I</text>

Commit message: Remove zener diode from ADC circuit
Parts:
- Z2: value MM3Z3V6T1G -> DNP
Changed lines of the file:
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@@
 <attribute name="VALUE" x="29.695" y="14.235" size="1.27" layer="27" rot="R270"/>
 </element>
-<element name="Z2" library="MM3Z3V6T1G" package="SOD2512X110N" value="MM3Z3V6T1G" x="28.9" y="19.9" smashed="yes" rot="R90">
+<element name="Z2" library="MM3Z3V6T1G" package="SOD2512X110N" value="DNP" x="28.9" y="19.9" smashed="yes" rot="R90">
 <attribute name="DESCRIPTION" value="ON Semiconductor MM3Z3V6T1G Zener Diode, 3.6V 5% 200 mW SMT 2-Pin SOD-323" x="28.9" y="19.9" size="1.778" layer="27" rot="R90" display="off"/>
 <attribute name="HEIGHT" value="1.1mm" x="28.9" y="19.9" size="1.778" layer="27" rot="R90" display="off"/>
@@
 <attribute name="MPN" value="MM3Z3V6T1G" x="28.9" y="19.9" size="1.778" layer="27" rot="R90" display="off"/>
 <attribute name="NAME" x="28.9" y="19.9" size="1.27" layer="25" rot="R90" align="center"/>
+<attribute name="POPULATE" value="0" x="28.9" y="19.9" size="1.778" layer="27" rot="R90" display="off"/>
 <attribute name="VALUE" x="28.9" y="19.9" size="1.27" layer="27" rot="R90" align="center"/>
 </element>
