File: openmv5/relay/relay.brd (EAGLE design)
At the start: 35.6 x 26.7 mm, 77 parts, among them IC1 TPS613222ADBVR, IC2 AP64060WU-7, IC3 LM321LVIDCKR, IC4 74LVC1G07GW,125, J1 OPENMV5-TOP, J2 1771088, K1 IMC03TS, K2 IMC03TS, Q1 SSM3J356R,LF, Q2 2N7002KW_R1_00001, Q3 2N7002KW_R1_00001, U1 74LVC1G17SE-7

Commit message: Remove zener diode from ADC circuit
Parts:
- Z2: value MM3Z3V6T1G -> DNP
Changed lines of the file:
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@@
 <attribute name="VALUE" x="29.695" y="14.235" size="1.27" layer="27" rot="R270"/>
 </element>
-<element name="Z2" library="MM3Z3V6T1G" package="SOD2512X110N" value="MM3Z3V6T1G" x="28.9" y="19.9" smashed="yes" rot="R90">
+<element name="Z2" library="MM3Z3V6T1G" package="SOD2512X110N" value="DNP" x="28.9" y="19.9" smashed="yes" rot="R90">
 <attribute name="DESCRIPTION" value="ON Semiconductor MM3Z3V6T1G Zener Diode, 3.6V 5% 200 mW SMT 2-Pin SOD-323" x="28.9" y="19.9" size="1.778" layer="27" rot="R90" display="off"/>
 <attribute name="HEIGHT" value="1.1mm" x="28.9" y="19.9" size="1.778" layer="27" rot="R90" display="off"/>
@@
 <attribute name="MPN" value="MM3Z3V6T1G" x="28.9" y="19.9" size="1.778" layer="27" rot="R90" display="off"/>
 <attribute name="NAME" x="28.9" y="19.9" size="1.27" layer="25" rot="R90" align="center"/>
+<attribute name="POPULATE" value="0" x="28.9" y="19.9" size="1.778" layer="27" rot="R90" display="off"/>
 <attribute name="VALUE" x="28.9" y="19.9" size="1.27" layer="27" rot="R90" align="center"/>
 </element>
