File: openmv5/poe/poe.sch (EAGLE design)
At the start: 47 parts, among them IC1 AG9905LP, J1 GMJXHT-MM-S-88, J2 OPENMV5-BOTTOM, T1 PT61018PEL

Commit message: Fix wrong inductor in PoE
Parts:
- L1, L2, L3, L4, L5, L6: MPN BBPY00100505102Y00 -> 2508051027Y1
Changed lines of the file:
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@@
 </part>
 <part name="L6" library="SparkFun-Coils" library_urn="urn:adsk.eagle:library:512" deviceset="INDUCTOR" device="-0805-3.3UH" package3d_urn="urn:adsk.eagle:package:37579/1" value="1K">
-<attribute name="MPN" value="BBPY00100505102Y00"/>
+<attribute name="MPN" value="2508051027Y1"/>
 </part>
 <part name="L4" library="SparkFun-Coils" library_urn="urn:adsk.eagle:library:512" deviceset="INDUCTOR" device="-0805-3.3UH" package3d_urn="urn:adsk.eagle:package:37579/1" value="1K">
-<attribute name="MPN" value="BBPY00100505102Y00"/>
+<attribute name="MPN" value="2508051027Y1"/>
 </part>
 <part name="L2" library="SparkFun-Coils" library_urn="urn:adsk.eagle:library:512" deviceset="INDUCTOR" device="-0805-3.3UH" package3d_urn="urn:adsk.eagle:package:37579/1" value="1K">
-<attribute name="MPN" value="BBPY00100505102Y00"/>
+<attribute name="MPN" value="2508051027Y1"/>
 </part>
 <part name="L5" library="SparkFun-Coils" library_urn="urn:adsk.eagle:library:512" deviceset="INDUCTOR" device="-0805-3.3UH" package3d_urn="urn:adsk.eagle:package:37579/1" value="1K">
-<attribute name="MPN" value="BBPY00100505102Y00"/>
+<attribute name="MPN" value="2508051027Y1"/>
 </part>
 <part name="L3" library="SparkFun-Coils" library_urn="urn:adsk.eagle:library:512" deviceset="INDUCTOR" device="-0805-3.3UH" package3d_urn="urn:adsk.eagle:package:37579/1" value="1K">
-<attribute name="MPN" value="BBPY00100505102Y00"/>
+<attribute name="MPN" value="2508051027Y1"/>
 </part>
 <part name="L1" library="SparkFun-Coils" library_urn="urn:adsk.eagle:library:512" deviceset="INDUCTOR" device="-0805-3.3UH" package3d_urn="urn:adsk.eagle:package:37579/1" value="1K">
-<attribute name="MPN" value="BBPY00100505102Y00"/>
+<attribute name="MPN" value="2508051027Y1"/>
 </part>
 <part name="C12" library="rcl" library_urn="urn:adsk.eagle:library:334" deviceset="C-EU" device="C1206" package3d_urn="urn:adsk.eagle:package:23618/2" value="1nF">
