File: openmv5/onsemi/ahdr.brd (EAGLE design)
At the start: 35.6 x 16.5 mm, 75 parts, among them IC1 AR0231AT7C00XUEA0-DRBR-E, IC2 TLV62568PDDCR, IC3 MIC5365-2.8YC5-TR, J1 DF12-36-DP, Q1 PMXB120EPEZ

Commit message: Update resistor value
Parts:
- R3: value 1K -> 10K
Changed lines of the file:
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@@
 <attribute name="VALUE" x="13.9065" y="3.5005" size="0.8128" layer="27" ratio="10" rot="R180"/>
 </element>
-<element name="R3" library="rcl" library_urn="urn:adsk.eagle:library:334" package="R0402" package3d_urn="urn:adsk.eagle:package:23547/3" value="1K" x="14.732" y="2.159" smashed="yes" rot="MR90">
-<attribute name="MPN" value="CRCW04021K00FKEDC" x="14.732" y="2.159" size="1.778" layer="28" rot="MR90" display="off"/>
+<element name="R3" library="rcl" library_urn="urn:adsk.eagle:library:334" package="R0402" package3d_urn="urn:adsk.eagle:package:23547/3" value="10K" x="14.732" y="2.159" smashed="yes" rot="MR90">
+<attribute name="MPN" value="AC0402FR-1310KL" x="14.732" y="2.159" size="1.778" layer="28" rot="MR90" display="off"/>
 <attribute name="NAME" x="15.367" y="1.524" size="1.27" layer="26" rot="MR90"/>
 <attribute name="POPULARITY" value="34" x="14.732" y="2.159" size="1.778" layer="28" rot="MR90" display="off"/>
