File: openmv5/driver/driver.brd (EAGLE design)
At the start: 35.6 x 26.7 mm, 87 parts, among them IC1 TPS613222ADBVR, IC2 AP64060WU-7, IC3 LM321LVIDCKR, IC4 74LVC1G07GW,125, IC5 DRV8876RGTR, IC6 DRV8876RGTR, J1 OPENMV5-TOP, J2 1771088, Q1 BUK6D120-60PX, U1 74LVC1G17SE-7

Commit message: Finish up driver shield
Parts:
- C16, C17: value EEV226M050S9GAA -> EMZR500ARA101MF80G; device EEV226M050S9GAA:CAPAE660X565N -> EMZR500ARA101MF80G:CAPAE660X820N
- moved JP2 5.90 mm to (7.00, 25.0), flipped to the top, turned to 0 degrees
- moved JP3 5.90 mm to (11.6, 21.3), flipped to the bottom, turned to 270 degrees
Routing:
- net P1_PWM_INT: track 14.7 -> 11.0 mm
- net P2_PWM_INT: track 14.1 -> 17.4 mm
- net P12_PWM: track 15.1 -> 16.1 mm
- net EXT_VIN_INT: track 46.2 -> 46.8 mm
- net GND: track 213.6 -> 213.3 mm, vias 33 -> 43
Other:
- board text added: "H"
- board text added: "L"
- board text removed: "MOD"

Commit message: Fix placement
Parts:
- moved JP8 0.20 mm to (25.6, 15.7)
Changed lines of the file:
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@@
 <text x="29" y="13" size="0.8128" layer="22" font="vector" ratio="22" rot="MR0">O</text>
 <text x="27.3" y="13" size="0.8128" layer="22" font="vector" ratio="22" rot="MR0">I</text>
-<text x="24" y="15.2" size="0.8128" layer="21" font="vector" ratio="22" rot="R180">mA</text>
+<text x="24.3" y="15.2" size="0.8128" layer="21" font="vector" ratio="22" rot="R180">mA</text>
 <text x="13.6" y="25.2" size="0.8128" layer="21" font="vector" ratio="20">PWR - 6V to 36V </text>
 <text x="13.6" y="24" size="0.8128" layer="21" font="vector" ratio="20">AIN - 0 to 5V or 4-20mA</text>
@@
 <attribute name="VALUE" x="30.8" y="16.5" size="1.27" layer="27" align="center"/>
 </element>
-<element name="JP8" library="SparkFun-Jumpers" library_urn="urn:adsk.eagle:library:528" package="SMT-JUMPER_2_NO_SILK" package3d_urn="urn:adsk.eagle:package:39279/1" value="JUMPER-SMT_2_NO_SILK" x="25.4" y="15.7" smashed="yes">
-<attribute name="NAME" x="25.4" y="16.843" size="0.6096" layer="25" font="vector" ratio="20" align="bottom-center"/>
-<attribute name="VALUE" x="25.4" y="14.557" size="0.6096" layer="27" font="vector" ratio="20" align="top-center"/>
+<element name="JP8" library="SparkFun-Jumpers" library_urn="urn:adsk.eagle:library:528" package="SMT-JUMPER_2_NO_SILK" package3d_urn="urn:adsk.eagle:package:39279/1" value="JUMPER-SMT_2_NO_SILK" x="25.6" y="15.7" smashed="yes">
+<attribute name="NAME" x="25.6" y="16.843" size="0.6096" layer="25" font="vector" ratio="20" align="bottom-center"/>
+<attribute name="VALUE" x="25.6" y="14.557" size="0.6096" layer="27" font="vector" ratio="20" align="top-center"/>
 </element>
 <element name="C9" library="sfe" package="0402-CAP" value="0.1uF" x="31.3" y="18.5" smashed="yes">
@@
 <via x="27.1" y="15.5" extent="1-16" drill="0.4064"/>
 <wire x1="27.2" y1="14.6" x2="26.75" y2="14.6" width="0.4064" layer="16"/>
-<wire x1="27.1" y1="15.5" x2="26.6" y2="15" width="0.4064" layer="1"/>
-<wire x1="26.6" y1="15" x2="26.6" y2="10.1" width="0.4064" layer="1"/>
+<wire x1="27.1" y1="15.5" x2="27.1" y2="14.3" width="0.4064" layer="1"/>
+<wire x1="27.1" y1="14.3" x2="26.6" y2="13.8" width="0.4064" layer="1"/>
+<wire x1="26.6" y1="13.8" x2="26.6" y2="10.1" width="0.4064" layer="1"/>
 <contactref element="D5" pad="2"/>
 <contactref element="R8" pad="2"/>
@@
 <contactref element="R4" pad="2"/>
 <contactref element="JP8" pad="2"/>
-<wire x1="25.8064" y1="15.7" x2="25.8064" y2="10.4" width="0.4064" layer="1"/>
-<wire x1="25.8064" y1="10.4" x2="25.35" y2="10.4" width="0.4064" layer="1"/>
-<wire x1="25.8064" y1="15.7" x2="25.8064" y2="16.0064" width="0.4064" layer="1"/>
-<wire x1="26.7" y1="16.9" x2="25.8064" y2="16.0064" width="0.4064" layer="1"/>
+<wire x1="26.0064" y1="15.7" x2="25.9064" y2="15.6" width="0.4064" layer="1"/>
+<wire x1="25.9064" y1="15.6" x2="25.9064" y2="10.4" width="0.4064" layer="1"/>
+<wire x1="25.9064" y1="10.4" x2="25.35" y2="10.4" width="0.4064" layer="1"/>
+<wire x1="26.0064" y1="15.7" x2="26.0064" y2="16.2064" width="0.4064" layer="1"/>
+<wire x1="26.7" y1="16.9" x2="26.0064" y2="16.2064" width="0.4064" layer="1"/>
 <wire x1="27.5" y1="18.65" x2="27.2" y2="18.65" width="0.4064" layer="1"/>
 <wire x1="27.2" y1="18.65" x2="26.7" y2="18.15" width="0.4064" layer="1"/>
@@
 <contactref element="JP8" pad="1"/>
 <contactref element="R11" pad="2"/>
-<wire x1="24.9936" y1="15.7" x2="25.0936" y2="15.8" width="0.4064" layer="1"/>
+<wire x1="25.1936" y1="15.7" x2="25.0936" y2="15.8" width="0.4064" layer="1"/>
 <wire x1="25.0936" y1="16.8436" x2="25.0936" y2="15.8" width="0.4064" layer="1"/>
 <wire x1="25.8" y1="17.55" x2="25.0936" y2="16.8436" width="0.4064" layer="1"/>
@@
 <via x="19.7" y="19.8" extent="1-16" drill="0.254"/>
 <wire x1="19.7" y1="19.8" x2="20.7" y2="20.8" width="0.254" layer="1"/>
-<wire x1="20.7" y1="20.8" x2="23.6" y2="20.8" width="0.254" layer="1"/>
-<via x="23.6" y="20.8" extent="1-16" drill="0.254"/>
-<wire x1="23.6" y1="20.8" x2="23.8" y2="20.8" width="0.254" layer="16"/>
+<wire x1="20.7" y1="20.8" x2="23.5" y2="20.8" width="0.254" layer="1"/>
+<via x="23.5" y="20.8" extent="1-16" drill="0.254"/>
+<wire x1="23.5" y1="20.8" x2="23.8" y2="20.8" width="0.254" layer="16"/>
 <wire x1="24.6" y1="19.8" x2="23.8" y2="19.8" width="0.254" layer="16"/>
 <wire x1="24.6" y1="19.8" x2="24.8" y2="19.6" width="0.254" layer="16"/>
@@
 <via x="10.1" y="19.8" extent="1-16" drill="0.254"/>
 <wire x1="10.1" y1="19.8" x2="11.1" y2="20.8" width="0.254" layer="1"/>
-<wire x1="11.1" y1="20.8" x2="14" y2="20.8" width="0.254" layer="1"/>
-<via x="14" y="20.8" extent="1-16" drill="0.254"/>
-<wire x1="14" y1="20.8" x2="14.2" y2="20.8" width="0.254" layer="16"/>
+<wire x1="11.1" y1="20.8" x2="13.9" y2="20.8" width="0.254" layer="1"/>
+<via x="13.9" y="20.8" extent="1-16" drill="0.254"/>
+<wire x1="13.9" y1="20.8" x2="14.2" y2="20.8" width="0.254" layer="16"/>
 <wire x1="15" y1="19.8" x2="14.2" y2="19.8" width="0.254" layer="16"/>
 <wire x1="15" y1="19.8" x2="15.2" y2="19.6" width="0.254" layer="16"/>

Commit message: Fix drc issues
Parts:
- moved D10 0.60 mm to (17.2, 21.8)
- moved D11 0.60 mm to (7.60, 21.8)
- moved D12 0.60 mm to (22.8, 21.8)
- moved D13 0.50 mm to (13.2, 21.7)
- moved FD3 0.42 mm to (6.70, 12.7)
- moved FD4 0.42 mm to (6.70, 12.7)
- moved FD2 0.36 mm to (29.6, 13.2)
- moved JP4 0.10 mm to (6.60, 8.50)
Routing:
- net GND: track 213.3 -> 215.3 mm
- net P8_PWM_INT: track 40.9 -> 41.5 mm

Commit message: Add servo shield
Other:
- board text added: "ADC P6"
- board text added: "FSYNC P10"
- board text removed: "ADC P11"
- board text removed: "FSYNC P11"
Changed lines of the file:
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@@
 <text x="32.4" y="2.8" size="0.8128" layer="22" font="vector" ratio="22" rot="MR270">GND</text>
 <text x="28.8" y="17.5" size="0.8128" layer="22" font="vector" ratio="22" rot="MR180">FSYNC
-P11</text>
+P10</text>
 <text x="11.9" y="12.6" size="0.8128" layer="21" font="vector" ratio="22">GND</text>
 <text x="9.4" y="12.6" size="0.8128" layer="21" font="vector" ratio="22">PWR</text>
@@
 <text x="32.4" y="5.3" size="0.8128" layer="22" font="vector" ratio="22" rot="MR270">VIN</text>
 <text x="5.6" y="9.9" size="0.8128" layer="22" font="vector" ratio="22" rot="MR90">ADC
-P11</text>
+P6</text>
 <text x="28.9" y="13" size="0.8128" layer="22" font="vector" ratio="22" rot="MR0">O</text>
 <text x="27.3" y="13" size="0.8128" layer="22" font="vector" ratio="22" rot="MR0">I</text>

Commit message: Remove zener diode from ADC circuit
Parts:
- Z2: value MM3Z3V6T1G -> DNP
Changed lines of the file:
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@@
 <attribute name="VALUE" x="29.395" y="14.435" size="1.27" layer="27" rot="R270"/>
 </element>
-<element name="Z2" library="MM3Z3V6T1G" package="SOD2512X110N" value="MM3Z3V6T1G" x="28.9" y="19.9" smashed="yes" rot="R90">
+<element name="Z2" library="MM3Z3V6T1G" package="SOD2512X110N" value="DNP" x="28.9" y="19.9" smashed="yes" rot="R90">
 <attribute name="DESCRIPTION" value="ON Semiconductor MM3Z3V6T1G Zener Diode, 3.6V 5% 200 mW SMT 2-Pin SOD-323" x="28.9" y="19.9" size="1.778" layer="27" rot="R90" display="off"/>
 <attribute name="HEIGHT" value="1.1mm" x="28.9" y="19.9" size="1.778" layer="27" rot="R90" display="off"/>
@@
 <attribute name="MPN" value="MM3Z3V6T1G" x="28.9" y="19.9" size="1.778" layer="27" rot="R90" display="off"/>
 <attribute name="NAME" x="28.9" y="19.9" size="1.27" layer="25" rot="R90" align="center"/>
+<attribute name="POPULATE" value="0" x="28.9" y="19.9" size="1.778" layer="27" rot="R90" display="off"/>
 <attribute name="VALUE" x="28.9" y="19.9" size="1.27" layer="27" rot="R90" align="center"/>
 </element>

Commit message: Update boards
Parts:
- removed Z3: MMSZ5231B-7-F, MMSZ5231B-7-F:SOD3716X145N
- added D14: CPDQT5V0HE-HF, CPDQT5V0HE-HF:CPDQT5V0HEHF
- D10: value CPDQT5V0HE-HF -> BAT54S_R1_00001; device CPDQT5V0HE-HF:CPDQT5V0HEHF -> BAT54S_R1_00001:SOT95P240X110-3N
- Z2: value DNP -> MMSZ5231B-7-F; device MM3Z3V6T1G:SOD2512X110N -> MMSZ5231B-7-F:SOD3716X145N
- moved D12 15.2 mm to (7.60, 21.8)
- moved Z2 12.3 mm to (23.1, 9.10), flipped to the bottom, turned to 0 degrees
- moved D10 11.6 mm to (28.8, 21.3), flipped to the top, turned to 0 degrees
- moved D13 9.60 mm to (22.8, 21.8)
- moved D11 9.60 mm to (17.2, 21.8)
- moved D5 1.64 mm to (29.6, 18.7)
- moved R4 0.71 mm to (28.0, 18.8), turned to 180 degrees
Connections:
- net AIN_INT: now also D10.3; no longer Z2.1
- net GND: now also D10.1, D14.2; no longer D10.2, Z3.2
- net P0_PWM: now also D13.1; no longer D12.1
- net P12_PWM: now also D14.1; no longer D13.1
- net P7_PWM: now also D11.1; no longer D10.1
- net P8_PWM: now also D12.1; no longer D11.1
- net SYNC_IN_INT: now also Z2.1; no longer Z3.1
- net VCC: now also D10.2
Routing:
- net VCC: track 69.7 -> 73.5 mm, vias 3 -> 4
- net GND: track 215.3 -> 212.1 mm, vias 43 -> 44
- net AIN_INT: track 7.92 -> 7.37 mm
Other:
- board text added: "5.11.23"
- board text removed: "4.17.23"
