File: openmv5/rt1060r1/rt1060r1.sch (EAGLE design)
At the start: 218 parts, among them CN1 S2B-PH-K-S(LF)(SN), IC1 LM66200DRLR, IC2 AP61300Z6-7, IC3 IS42S16160G-6BL, IC4 ATECC608B-MAHDA-T, IC5 IS25LP064D-JKLE-TR, IC6 IS25LP128F-JKLE-TR, IC7 MXC4005XC, IC8 MIMXRT106FCVL5B, IC9 KSZ8081RNDCA-TR, J1 USB4105-GF-A, J2 DNP, J3 DNP, J4 DF12-36-DS, J5 USD-1040310811, J6 DNP, J7 DNP, J8 3221-10-0300-00, M1 9774030151R, M2 9774030151R, Q1 2N7002KW_R1_00001, Q2 2N7002KW_R1_00001, Q3 2N7002KW_R1_00001, Q4 2N7002KW_R1_00001, Q5 2N7002KW_R1_00001, Q6 PMXB120EPEZ, U1 MIC5365-3.3YMT-TZ, U2 BQ24075RGTR, U3 LBEE5KL1DX-883, Y1 SC32S-7PF20PPM, Y2 XRCGB24M000F3M00R0

Commit message: Fix labels
Parts:
- IC8: DESCRIPTION (none) -> Processors - Application Specialized MIMXRT106FCVL5B/LFBGA1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; MANUFACTURER_PART_NUMBER (none) -> MIMXRT106FCVL5B; MOUSER_PART_NUMBER (none) -> 771-MIMXRT106FCVL5B; MOUSER_PRICE-STOCK (none) -> https://www.mouser.co.uk/ProductDetail/NXP-Semiconductors/M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
Other:
- note added: "* CKE is pulled down by 100K on the RT1062"
- note removed: "* CKE is pulled down by 100K on the RT1052"
Changed lines of the file:
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@@
 <part name="P+1" library="SparkFun" deviceset="VCC" device=""/>
 <part name="IC8" library="MIMXRT1052DVL6B" deviceset="MIMXRT1052DVL6B" device="" value="MIMXRT106FCVL5B">
+<attribute name="DESCRIPTION" value="Processors - Application Specialized MIMXRT106FCVL5B/LFBGA196///STANDARD MARKING * TRAY"/>
+<attribute name="MANUFACTURER_PART_NUMBER" value="MIMXRT106FCVL5B"/>
+<attribute name="MOUSER_PART_NUMBER" value="771-MIMXRT106FCVL5B"/>
+<attribute name="MOUSER_PRICE-STOCK" value="https://www.mouser.co.uk/ProductDetail/NXP-Semiconductors/MIMXRT106FCVL5B"/>
 <attribute name="MPN" value="MIMXRT106FCVL5B"/>
 </part>
@@
 <wire x1="208.28" y1="421.64" x2="106.68" y2="421.64" width="0.1524" layer="150" style="longdash"/>
 <wire x1="106.68" y1="421.64" x2="106.68" y2="429.26" width="0.1524" layer="150" style="longdash"/>
-<text x="109.22" y="424.18" size="2.54" layer="150" font="vector" ratio="20">* CKE is pulled down by 100K on the RT1052</text>
+<text x="109.22" y="424.18" size="2.54" layer="150" font="vector" ratio="20">* CKE is pulled down by 100K on the RT1062</text>
 <wire x1="703.58" y1="441.96" x2="858.52" y2="441.96" width="0.1524" layer="150" style="longdash"/>
 <wire x1="858.52" y1="441.96" x2="858.52" y2="434.34" width="0.1524" layer="150" style="longdash"/>
